File: PCB/configurations.kicad_sch (KiCad schematic)
At the start: 16 parts, among them SW1 SW_Push, U1 XC7A50T-FGG484, U7 MT25QL128ABA1EW7-0SIT

Commit message: cleaning up USB-C, switching some of the decoupling and assigning a bunch of footprints
Parts:
- C112: footprint (none) -> Capacitor_SMD:C_0402_1005Metric
Changed lines of the file:
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@@
 			)
 		)
-		(property "Footprint" ""
+		(property "Footprint" "Capacitor_SMD:C_0402_1005Metric"
 			(at 335.28 143.8148 0)
 			(effects
