File: PCB/configurations.kicad_sch (KiCad schematic)
At the start: 16 parts, among them SW1 SW_Push, U1 XC7A50T-FGG484, U7 MT25QL128ABA1EW7-0SIT

Commit message: forgot to add decouping to my banks
Parts:
- added C147: 47u, Capacitor_SMD:C_1206_3216Metric, symbol Device:C
- added C148, C149: 4u7, Capacitor_SMD:C_0603_1608Metric, symbol Device:C
- added C150, C151, C152, C153: 470n, Capacitor_SMD:C_0201_0603Metric, symbol Device:C
Connections:
- net +3V3: now also C147.1, C148.1, C149.1, C150.1, C151.1, C152.1, C153.1
- net GND: now also C147.2, C148.2, C149.2, C150.2, C151.2, C152.2, C153.2
Other:
- moved on the sheet: D1, R22, R24, SW1

Commit message: fixed my decoupling because I'm better than the datasheet
Parts:
- removed C148, C149: 4u7, Capacitor_SMD:C_0603_1608Metric, symbol Device:C
- removed C152, C153: 470n, Capacitor_SMD:C_0201_0603Metric, symbol Device:C
Other:
- moved on the sheet: C150, C151

Commit message: adding return via's and cleaning up the schematic a bit!
Other:
- moved on the sheet: D1, R22, R24, SW1
Changed lines of the file:
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@@
 	(text "< Manual configuration reset, it's a devboard so why not"
 		(exclude_from_sim no)
-		(at 147.828 87.63 0)
+		(at 147.828 82.55 0)
 		(effects
 			(font
@@
 	(text "< DONE sinks current, LED turns off when done"
 		(exclude_from_sim no)
-		(at 122.428 52.324 0)
+		(at 122.428 47.244 0)
 		(effects
 			(font
@@
 	)
 	(junction
-		(at 93.98 86.36)
+		(at 93.98 81.28)
 		(diameter 0)
 		(color 0 0 0 0)
@@
 	(wire
 		(pts
-			(xy 93.98 86.36) (xy 102.87 86.36)
+			(xy 93.98 81.28) (xy 102.87 81.28)
 		)
 		(stroke
@@
 	(wire
 		(pts
-			(xy 93.98 73.66) (xy 93.98 76.2)
+			(xy 93.98 68.58) (xy 93.98 71.12)
 		)
 		(stroke
@@
 	(wire
 		(pts
-			(xy 85.09 52.07) (xy 90.17 52.07)
+			(xy 85.09 46.99) (xy 90.17 46.99)
 		)
 		(stroke
@@
 	(wire
 		(pts
-			(xy 115.57 86.36) (xy 113.03 86.36)
+			(xy 115.57 81.28) (xy 113.03 81.28)
 		)
 		(stroke
@@
 	(wire
 		(pts
-			(xy 81.28 86.36) (xy 93.98 86.36)
+			(xy 81.28 81.28) (xy 93.98 81.28)
 		)
 		(stroke
@@
 	(wire
 		(pts
-			(xy 118.11 52.07) (xy 110.49 52.07)
+			(xy 118.11 46.99) (xy 110.49 46.99)
 		)
 		(stroke
@@
 	(wire
 		(pts
-			(xy 97.79 52.07) (xy 102.87 52.07)
+			(xy 97.79 46.99) (xy 102.87 46.99)
 		)
 		(stroke
@@
 	(wire
 		(pts
-			(xy 93.98 83.82) (xy 93.98 86.36)
+			(xy 93.98 78.74) (xy 93.98 81.28)
 		)
 		(stroke
@@
 	)
 	(label "PROG_B"
-		(at 81.28 86.36 0)
+		(at 81.28 81.28 0)
 		(effects
 			(font
@@
 	)
 	(label "DONE"
-		(at 118.11 52.07 180)
+		(at 118.11 46.99 180)
 		(effects
 			(font
@@
 	(symbol
 		(lib_id "power:GND")
-		(at 115.57 86.36 0)
+		(at 115.57 81.28 0)
 		(unit 1)
 		(body_style 1)
@@
 		(fields_autoplaced yes)
 		(property "Reference" "#PWR07"
-			(at 115.57 92.71 0)
+			(at 115.57 87.63 0)
 			(hide yes)
 			(show_name no)
@@
 		)
 		(property "Value" "GND"
-			(at 115.57 91.44 0)
+			(at 115.57 86.36 0)
 			(show_name no)
 			(do_not_autoplace no)
@@
 		)
 		(property "Footprint" ""
-			(at 115.57 86.36 0)
+			(at 115.57 81.28 0)
 			(hide yes)
 			(show_name no)
@@
 		)
 		(property "Datasheet" ""
-			(at 115.57 86.36 0)
+			(at 115.57 81.28 0)
 			(hide yes)
 			(show_name no)
@@
 		)
 		(property "Description" "Power symbol creates a global label with name \"GND\" , ground"
-			(at 115.57 86.36 0)
+			(at 115.57 81.28 0)
 			(hide yes)
 			(show_name no)
@@
 	(symbol
 		(lib_id "Switch:SW_Push")
-		(at 107.95 86.36 0)
+		(at 107.95 81.28 0)
 		(unit 1)
 		(body_style 1)
@@
 		(fields_autoplaced yes)
 		(property "Reference" "SW1"
-			(at 107.95 78.74 0)
+			(at 107.95 73.66 0)
 			(show_name no)
 			(do_not_autoplace no)
@@
 		)
 		(property "Value" "SW_Push"
-			(at 107.95 81.28 0)
+			(at 107.95 76.2 0)
 			(show_name no)
 			(do_not_autoplace no)
@@
 		)
 		(property "Footprint" "Button_Switch_SMD:SW_SPST_TS-1088-xR020"
-			(at 107.95 81.28 0)
+			(at 107.95 76.2 0)
 			(hide yes)
 			(show_name no)
@@
 		)
 		(property "Datasheet" ""
-			(at 107.95 81.28 0)
+			(at 107.95 76.2 0)
 			(hide yes)
 			(show_name no)
@@
 		)
 		(property "Description" "Push button switch, generic, two pins"
-			(at 107.95 86.36 0)
+			(at 107.95 81.28 0)
 			(hide yes)
 			(show_name no)
@@
 		)
 		(property "MPN" "TS-1088-AR02016"
-			(at 107.95 86.36 0)
+			(at 107.95 81.28 0)
 			(hide yes)
 			(show_name no)
@@
 		)
 		(property "LCSC" "C720477"
-			(at 107.95 86.36 0)
+			(at 107.95 81.28 0)
 			(hide yes)
 			(show_name no)
@@
 	(symbol
 		(lib_id "Device:LED")
-		(at 93.98 52.07 180)
+		(at 93.98 46.99 180)
 		(unit 1)
 		(body_style 1)
@@
 		(dnp no)
 		(property "Reference" "D1"
-			(at 93.98 48.006 0)
+			(at 93.98 42.926 0)
 			(show_name no)
 			(do_not_autoplace no)
@@
 		)
 		(property "Value" "KT-0805Y"
-			(at 93.98 45.466 0)
+			(at 93.98 40.386 0)
 			(show_name no)
 			(do_not_autoplace no)
@@
 		)
 		(property "Footprint" "LED_SMD:LED_0805_2012Metric"
-			(at 93.98 52.07 0)
+			(at 93.98 46.99 0)
 			(hide yes)
 			(show_name no)
@@
 		)
 		(property "Datasheet" ""
-			(at 93.98 52.07 0)
+			(at 93.98 46.99 0)
 			(hide yes)
 			(show_name no)
@@
 		)
 		(property "Description" "Light emitting diode"
-			(at 93.98 52.07 0)
+			(at 93.98 46.99 0)
 			(hide yes)
 			(show_name no)
@@
 		)
 		(property "Sim.Pins" "1=K 2=A"
-			(at 93.98 52.07 0)
+			(at 93.98 46.99 0)
 			(hide yes)
 			(show_name no)
@@
 		)
 		(property "MPN" "KT-0805Y"
-			(at 93.98 52.07 0)
+			(at 93.98 46.99 0)
 			(hide yes)
 			(show_name no)
@@
 		)
 		(property "LCSC" "C2296"
-			(at 93.98 52.07 0)
+			(at 93.98 46.99 0)
 			(hide yes)
 			(show_name no)
@@
 	(symbol
 		(lib_id "power:+3V3")
-		(at 93.98 73.66 0)
+		(at 93.98 68.58 0)
 		(unit 1)
 		(body_style 1)
@@
 		(dnp no)
 		(property "Reference" "#PWR05"
-			(at 93.98 77.47 0)
+			(at 93.98 72.39 0)
 			(hide yes)
 			(show_name no)
@@
 		)
 		(property "Value" "+3V3"
-			(at 93.472 69.596 0)
+			(at 93.472 64.516 0)
 			(show_name no)
 			(do_not_autoplace no)
@@
 		)
 		(property "Footprint" ""
-			(at 93.98 73.66 0)
+			(at 93.98 68.58 0)
 			(hide yes)
 			(show_name no)
@@
 		)
 		(property "Datasheet" ""
-			(at 93.98 73.66 0)
+			(at 93.98 68.58 0)
 			(hide yes)
 			(show_name no)
@@
 		)
 		(property "Description" "Power symbol creates a global label with name \"+3V3\""
-			(at 93.98 73.66 0)
+			(at 93.98 68.58 0)
 			(hide yes)
 			(show_name no)
@@
 	(symbol
 		(lib_id "Device:R")
-		(at 93.98 80.01 0)
+		(at 93.98 74.93 0)
 		(unit 1)
 		(body_style 1)
@@
 		(fields_autoplaced yes)
 		(property "Reference" "R22"
-			(at 96.52 78.7399 0)
+			(at 96.52 73.6599 0)
 			(show_name no)
 			(do_not_autoplace no)
@@
 		)
 		(property "Value" "4k7"
-			(at 96.52 81.2799 0)
+			(at 96.52 76.1999 0)
 			(show_name no)
 			(do_not_autoplace no)
@@
 		)
 		(property "Footprint" "Resistor_SMD:R_0402_1005Metric"
-			(at 92.202 80.01 90)
+			(at 92.202 74.93 90)
 			(hide yes)
 			(show_name no)
@@
 		)
 		(property "Datasheet" ""
-			(at 93.98 80.01 0)
+			(at 93.98 74.93 0)
 			(hide yes)
 			(show_name no)
@@
 		)
 		(property "Description" "Resistor"
-			(at 93.98 80.01 0)
+			(at 93.98 74.93 0)
 			(hide yes)
 			(show_name no)
@@
 	(symbol
 		(lib_id "Device:R")
-		(at 106.68 52.07 270)
+		(at 106.68 46.99 270)
 		(mirror x)
 		(unit 1)
@@
 		(fields_autoplaced yes)
 		(property "Reference" "R24"
-			(at 106.68 45.72 90)
+			(at 106.68 40.64 90)
 			(show_name no)
 			(do_not_autoplace no)
@@
 		)
 		(property "Value" "1k"
-			(at 106.68 48.26 90)
+			(at 106.68 43.18 90)
 			(show_name no)
 			(do_not_autoplace no)
@@
 		)
 		(property "Footprint" "Resistor_SMD:R_0402_1005Metric"
-			(at 106.68 53.848 90)
+			(at 106.68 48.768 90)
 			(hide yes)
 			(show_name no)
@@
 		)
 		(property "Datasheet" ""
-			(at 106.68 52.07 0)
+			(at 106.68 46.99 0)
 			(hide yes)
 			(show_name no)
@@
 		)
 		(property "Description" "Resistor"
-			(at 106.68 52.07 0)
+			(at 106.68 46.99 0)
 			(hide yes)
 			(show_name no)
@@
 	(symbol
 		(lib_id "power:+3V3")
-		(at 85.09 52.07 0)
+		(at 85.09 46.99 0)
 		(mirror y)
 		(unit 1)
@@
 		(fields_autoplaced yes)
 		(property "Reference" "#PWR057"
-			(at 85.09 55.88 0)
+			(at 85.09 50.8 0)
 			(hide yes)
 			(show_name no)
@@
 		)
 		(property "Value" "+3V3"
-			(at 85.09 46.99 0)
+			(at 85.09 41.91 0)
 			(show_name no)
 			(do_not_autoplace no)
@@
 		)
 		(property "Footprint" ""
-			(at 85.09 52.07 0)
+			(at 85.09 46.99 0)
 			(hide yes)
 			(show_name no)
@@
 		)
 		(property "Datasheet" ""
-			(at 85.09 52.07 0)
+			(at 85.09 46.99 0)
 			(hide yes)
 			(show_name no)
@@
 		)
 		(property "Description" "Power symbol creates a global label with name \"+3V3\""
-			(at 85.09 52.07 0)
+			(at 85.09 46.99 0)
 			(hide yes)
 			(show_name no)
