File: PCB/ethernet.kicad_sch (KiCad schematic)
At the start: 39 parts, among them J5 RJ45_Hanrun_HR911105A_Horizon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, SW2 SW_Push, U13 LAN8710A-EZC-TR, Y1 50MHz

Commit message: cleaning up USB-C, switching some of the decoupling and assigning a bunch of footprints
Parts:
- C126, C130, C132, C133, C135, C136, C137, C138: footprint (none) -> Capacitor_SMD:C_0402_1005Metric
- FB4: footprint (none) -> Inductor_SMD:L_0805_2012Metric
Changed lines of the file:
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@@
 			)
 		)
-		(property "Footprint" ""
+		(property "Footprint" "Capacitor_SMD:C_0402_1005Metric"
 			(at 128.27 209.8548 0)
 			(effects
@@
 			)
 		)
-		(property "Footprint" ""
+		(property "Footprint" "Inductor_SMD:L_0805_2012Metric"
 			(at 140.97 62.738 90)
 			(effects
@@
 			)
 		)
-		(property "Footprint" ""
+		(property "Footprint" "Capacitor_SMD:C_0402_1005Metric"
 			(at 253.6952 163.83 0)
 			(effects
@@
 			)
 		)
-		(property "Footprint" ""
+		(property "Footprint" "Capacitor_SMD:C_0402_1005Metric"
 			(at 243.5352 163.83 0)
 			(effects
@@
 			)
 		)
-		(property "Footprint" ""
+		(property "Footprint" "Capacitor_SMD:C_0402_1005Metric"
 			(at 274.0152 163.83 0)
 			(effects
@@
 			)
 		)
-		(property "Footprint" ""
+		(property "Footprint" "Capacitor_SMD:C_0402_1005Metric"
 			(at 128.27 222.5548 0)
 			(effects
@@
 			)
 		)
-		(property "Footprint" ""
+		(property "Footprint" "Capacitor_SMD:C_0402_1005Metric"
 			(at 113.9952 71.12 0)
 			(effects
@@
 			)
 		)
-		(property "Footprint" ""
+		(property "Footprint" "Capacitor_SMD:C_0402_1005Metric"
 			(at 180.0352 71.12 0)
 			(effects
@@
 			)
 		)
-		(property "Footprint" ""
+		(property "Footprint" "Capacitor_SMD:C_0402_1005Metric"
 			(at 263.8552 163.83 0)
 			(effects

Commit message: even more footprints
Parts:
- C141: footprint (none) -> Capacitor_SMD:C_0402_1005Metric
Changed lines of the file:
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@@
 			)
 		)
-		(property "Footprint" ""
+		(property "Footprint" "Capacitor_SMD:C_0402_1005Metric"
 			(at 171.1452 96.52 0)
 			(effects

Commit message: adding some MPN's in, searching for ethernet RJ45's
Other:
- note added: "https://jlcpcb.com/partdetail/HDGC-RJ45_DB101PWB/C2936176"
- note added: "https://jlcpcb.com/partdetail/Heling-MJ88B_B011_RVL11P/C501462"
- note added: "https://jlcpcb.com/partdetail/Heling-MJ88_B011XRVS1/C501464"
- note added: "rj45 recessed lcsc"
Changed lines of the file:
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@@
 		(members "JTAG_TCK" "JTAG_TDI" "JTAG_TDO" "JTAG_TMS")
+	)
+	(text "rj45 recessed lcsc"
+		(exclude_from_sim no)
+		(at 286.766 180.34 0)
+		(effects
+			(font
+				(size 1.27 1.27)
+			)
+		)
 	)
 	(text "100 Mbps, RMII Ethernet!"
@@
 		)
 	)
+	(text "https://jlcpcb.com/partdetail/HDGC-RJ45_DB101PWB/C2936176"
+		(exclude_from_sim no)
+		(at 308.102 187.452 0)
+		(effects
+			(font
+				(size 1.27 1.27)
+			)
+		)
+	)
 	(text "< Internal pullup!"
 		(exclude_from_sim no)
@@
 		(effects
 			(font
+				(size 1.27 1.27)
+			)
+		)
+	)
+	(text "https://jlcpcb.com/partdetail/Heling-MJ88_B011XRVS1/C501464"
+		(exclude_from_sim no)
+		(at 309.88 200.66 0)
+		(effects
+			(font
+				(size 1.27 1.27)
+			)
+		)
+	)
+	(text "https://jlcpcb.com/partdetail/Heling-MJ88B_B011_RVL11P/C501462"
+		(exclude_from_sim no)
+		(at 308.864 193.548 0)
+		(effects
+			(font

Commit message: working on a new ethernet connector
Parts:
- added J3: MJ88-B011-HLSV6-P, easyeda2kicad:RJ45-SMD_MJ88-B011-HLSV6-P, symbol easyeda2kicad:MJ88-B011-HLSV6-P
Other:
- note removed: "https://jlcpcb.com/partdetail/HDGC-RJ45_DB101PWB/C2936176"
- note removed: "https://jlcpcb.com/partdetail/Heling-MJ88B_B011_RVL11P/C501462"
- note removed: "https://jlcpcb.com/partdetail/Heling-MJ88_B011XRVS1/C501464"
- note removed: "rj45 recessed lcsc"
Changed lines of the file:
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@@
 		(members "JTAG_TCK" "JTAG_TDI" "JTAG_TDO" "JTAG_TMS")
 	)
-	(text "rj45 recessed lcsc"
-		(exclude_from_sim no)
-		(at 286.766 180.34 0)
-		(effects
-			(font
-				(size 1.27 1.27)
-			)
-		)
-	)
 	(text "100 Mbps, RMII Ethernet!"
 		(exclude_from_sim no)
@@
 		)
 	)
-	(text "https://jlcpcb.com/partdetail/HDGC-RJ45_DB101PWB/C2936176"
-		(exclude_from_sim no)
-		(at 308.102 187.452 0)
-		(effects
-			(font
-				(size 1.27 1.27)
-			)
-		)
-	)
 	(text "< Internal pullup!"
 		(exclude_from_sim no)
@@
 		)
 	)
-	(text "https://jlcpcb.com/partdetail/Heling-MJ88_B011XRVS1/C501464"
-		(exclude_from_sim no)
-		(at 309.88 200.66 0)
-		(effects
-			(font
-				(size 1.27 1.27)
-			)
-		)
-	)
-	(text "https://jlcpcb.com/partdetail/Heling-MJ88B_B011_RVL11P/C501462"
-		(exclude_from_sim no)
-		(at 308.864 193.548 0)
-		(effects
-			(font
-				(size 1.27 1.27)
-			)
-		)
-	)
 	(text "< Driving the 3V3 analog rail"
 		(exclude_from_sim no)
@@
 					(unit 1)
 				)
+			)
+		)
+	)
+	(symbol
+		(lib_id "easyeda2kicad:MJ88-B011-HLSV6-P")
+		(at 313.69 214.63 270)
+		(unit 1)
+		(exclude_from_sim no)
+		(in_bom yes)
+		(on_board yes)
+		(dnp no)
+		(fields_autoplaced yes)
+		(property "Reference" "J3"
+			(at 313.69 196.85 90)
+			(effects
+				(font
+					(size 1.27 1.27)
+				)
+			)
+		)
+		(property "Value" "MJ88-B011-HLSV6-P"
+			(at 313.69 199.39 90)
+			(effects
+				(font
+					(size 1.27 1.27)
+				)
+			)
+		)
+		(property "Footprint" "easyeda2kicad:RJ45-SMD_MJ88-B011-HLSV6-P"
+			(at 343.154 214.884 0)
+			(effects
+				(font
+					(size 1.27 1.27)
+				)
+				(hide yes)
+			)
+		)
+		(property "Datasheet" ""
+			(at 313.69 214.63 0)
+			(effects
+				(font
+					(size 1.27 1.27)
+				)
+				(hide yes)
+			)
+		)
+		(property "Description" ""
+			(at 313.69 214.63 0)
+			(effects
+				(font
+					(size 1.27 1.27)
+				)
+				(hide yes)
+			)
+		)
+		(property "LCSC Part" "C501463"
+			(at 340.614 214.884 0)
+			(effects
+				(font
+					(size 1.27 1.27)
+				)
+				(hide yes)
+			)
+		)
+		(pin "8"
+		)
+		(pin "4"
+		)
+		(pin "1"
+		)
+		(pin "7"
+		)
+		(pin "6"
+		)
+		(pin "9"
+		)
+		(pin "2"
+		)
+		(pin "5"
+		)
+		(pin "10"
+		)
+		(pin "3"
+		)
+		(instances
+			(project ""
+				(path "/ed0095eb-57a0-4856-9ac4-7b40bd214a3a/09aa8758-c80d-4d7c-89ed-08037b84af81"
+					(reference "J3")
+					(unit 1)
+				)

Commit message: removing ethernet, out of scope ;)
Parts:
- removed C126, C130, C141: 1u, Capacitor_SMD:C_0402_1005Metric, symbol Device:C
- removed C127, C128, C129, C131, C134: 100n, Capacitor_SMD:C_0402_1005Metric, symbol Device:C
- removed C132, C133: 18p, Capacitor_SMD:C_0402_1005Metric, symbol Device:C
- removed C135, C136, C137, C138: 10p, Capacitor_SMD:C_0402_1005Metric, symbol Device:C
- removed C140: 470p, Capacitor_SMD:C_0603_1608Metric, symbol Device:C
- removed FB4: 120@100MHz, Inductor_SMD:L_0805_2012Metric, symbol Device:FerriteBead_Small
- removed J3: MJ88-B011-HLSV6-P, easyeda2kicad:RJ45-SMD_MJ88-B011-HLSV6-P, symbol easyeda2kicad:MJ88-B011-HLSV6-P
- removed J5: RJ45_Hanrun_HR911105A_Horizontal, Connector_RJ:RJ45_Hanrun_HR911105A_Horizontal, symbol Connector:RJ45_Hanrun_HR911105A_Horizontal
- removed R63: 12k, Resistor_SMD:R_0402_1005Metric, symbol Device:R
- removed R64, R69: 4k7, Resistor_SMD:R_0402_1005Metric, symbol Device:R
- removed R65, R68: 10k, Resistor_SMD:R_0402_1005Metric, symbol Device:R
- removed R66, R67: 1k, Resistor_SMD:R_0402_1005Metric, symbol Device:R
- removed R70: 1M, Resistor_SMD:R_0402_1005Metric, symbol Device:R
- removed R71, R72, R73, R74: 49.9, Resistor_SMD:R_0402_1005Metric, symbol Device:R
- removed R78, R79, R80, R81, R82, R83, R84: 22, Resistor_SMD:R_0402_1005Metric, symbol Device:R_Small
- removed SW2: SW_Push, Button_Switch_SMD:SW_SPST_TS-1088-xR020, symbol Switch:SW_Push
- removed U13: LAN8710A-EZC-TR, Package_DFN_QFN:QFN-32-1EP_5x5mm_P0.5mm_EP3.3x3.3mm_ThermalVias, symbol FPGA Accelerator:LAN8710A
- removed Y1: 50MHz, Crystal:Crystal_SMD_2520-4Pin_2.5x2.0mm, symbol Device:Crystal_GND24
Connections:
- no-connect marks 6 -> 0
Other:
- note removed: "100 Mbps, RMII Ethernet!"
- note removed: "100 ohm termination, and optional EMI shunts!"
- note removed: "< Driving the 3V3 analog rail"
- note removed: "< Internal pullup!"
- note removed: "< LED's are pulled high and become active-low"
