File: PCB/usb.kicad_sch (KiCad schematic)
At the start: 52 parts, among them J2 Conn_ARM_SWD_TagConnect_TC2030, J4 TYPE-C-31-M-12, U10 FT2232HQ, U3 TPD2EUSB30, U4 TPD2EUSB30, U6 TPD2EUSB30, U8 TPS62132, U9 M93C56-WMN6TP, Y2 12MHz

Commit message: cleaning up USB-C, switching some of the decoupling and assigning a bunch of footprints
Parts:
- added C124: 4u7, symbol Device:C
- C87: value 10u -> 4u7
Connections:
- net +VBUS: now also C124.1
- net GND: now also C124.2
Other:
- moved on the sheet: C87, C88, C89, C90, C91, C92, L5, R50, U3, U8

Commit message: even more footprints
Parts:
- C124, C92, C96, C97: footprint (none) -> Capacitor_SMD:C_0402_1005Metric
- C87: footprint (none) -> Capacitor_SMD:C_0603_1608Metric
Other:
- moved on the sheet: C87
Changed lines of the file:
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@@
 	(wire
 		(pts
-			(xy 78.74 30.48) (xy 78.74 27.94)
+			(xy 78.74 31.75) (xy 78.74 27.94)
 		)
 		(stroke
@@
 	(wire
 		(pts
-			(xy 78.74 38.1) (xy 78.74 40.64)
+			(xy 78.74 39.37) (xy 78.74 43.18)
 		)
 		(stroke
@@
 	(wire
 		(pts
-			(xy 105.41 41.91) (xy 105.41 40.64)
+			(xy 105.41 43.18) (xy 105.41 40.64)
 		)
 		(stroke
@@
 	(symbol
 		(lib_id "Device:C")
-		(at 78.74 34.29 0)
+		(at 78.74 35.56 0)
 		(unit 1)
 		(exclude_from_sim no)
@@
 		(dnp no)
 		(property "Reference" "C87"
-			(at 79.756 31.242 0)
+			(at 79.756 32.512 0)
 			(effects
 				(font
@@
 		)
 		(property "Value" "4u7"
-			(at 79.756 37.338 0)
+			(at 79.756 38.608 0)
 			(effects
 				(font
@@
 			)
 		)
-		(property "Footprint" ""
-			(at 79.7052 38.1 0)
+		(property "Footprint" "Capacitor_SMD:C_0603_1608Metric"
+			(at 79.7052 39.37 0)
 			(effects
 				(font
@@
 		)
 		(property "Datasheet" "~"
-			(at 78.74 34.29 0)
+			(at 78.74 35.56 0)
 			(effects
 				(font
@@
 		)
 		(property "Description" "Unpolarized capacitor"
-			(at 78.74 34.29 0)
+			(at 78.74 35.56 0)
 			(effects
 				(font
@@
 			)
 		)
-		(property "Footprint" ""
+		(property "Footprint" "Capacitor_SMD:C_0402_1005Metric"
 			(at 97.4852 38.1 0)
 			(effects
@@
 			)
 		)
-		(property "Footprint" ""
+		(property "Footprint" "Capacitor_SMD:C_0402_1005Metric"
 			(at 111.76 237.7948 0)
 			(effects
@@
 	(symbol
 		(lib_id "power:GND")
-		(at 78.74 40.64 0)
+		(at 78.74 43.18 0)
 		(unit 1)
 		(exclude_from_sim no)
@@
 		(dnp no)
 		(property "Reference" "#PWR0153"
-			(at 78.74 46.99 0)
+			(at 78.74 49.53 0)
 			(effects
 				(font
@@
 		)
 		(property "Value" "GND"
-			(at 78.74 45.212 0)
+			(at 78.74 47.752 0)
 			(effects
 				(font
@@
 		)
 		(property "Footprint" ""
-			(at 78.74 40.64 0)
+			(at 78.74 43.18 0)
 			(effects
 				(font
@@
 		)
 		(property "Datasheet" ""
-			(at 78.74 40.64 0)
+			(at 78.74 43.18 0)
 			(effects
 				(font
@@
 		)
 		(property "Description" "Power symbol creates a global label with name \"GND\" , ground"
-			(at 78.74 40.64 0)
+			(at 78.74 43.18 0)
 			(effects
 				(font
@@
 			)
 		)
-		(property "Footprint" ""
+		(property "Footprint" "Capacitor_SMD:C_0402_1005Metric"
 			(at 111.76 247.9548 0)
 			(effects
@@
 			)
 		)
-		(property "Footprint" ""
+		(property "Footprint" "Capacitor_SMD:C_0402_1005Metric"
 			(at 195.2752 48.26 0)
 			(effects
@@
 	(symbol
 		(lib_id "power:GND")
-		(at 105.41 41.91 0)
+		(at 105.41 43.18 0)
 		(unit 1)
 		(exclude_from_sim no)
@@
 		(dnp no)
 		(property "Reference" "#PWR093"
-			(at 105.41 48.26 0)
+			(at 105.41 49.53 0)
 			(effects
 				(font
@@
 		)
 		(property "Value" "GND"
-			(at 105.41 46.228 0)
+			(at 105.41 47.752 0)
 			(effects
 				(font
@@
 		)
 		(property "Footprint" ""
-			(at 105.41 41.91 0)
+			(at 105.41 43.18 0)
 			(effects
 				(font
@@
 		)
 		(property "Datasheet" ""
-			(at 105.41 41.91 0)
+			(at 105.41 43.18 0)
 			(effects
 				(font
@@
 		)
 		(property "Description" "Power symbol creates a global label with name \"GND\" , ground"
-			(at 105.41 41.91 0)
+			(at 105.41 43.18 0)
 			(effects
 				(font

Commit message: fixing a bunch of footprints to standardize
Parts:
- C124: footprint Capacitor_SMD:C_0402_1005Metric -> Capacitor_SMD:C_0603_1608Metric
- C92: footprint Capacitor_SMD:C_0402_1005Metric -> Capacitor_SMD:C_1206_3216Metric
Changed lines of the file:
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@@
 			)
 		)
-		(property "Footprint" "Capacitor_SMD:C_0402_1005Metric"
+		(property "Footprint" "Capacitor_SMD:C_0603_1608Metric"
 			(at 97.4852 38.1 0)
 			(effects
@@
 			)
 		)
-		(property "Footprint" "Capacitor_SMD:C_0402_1005Metric"
+		(property "Footprint" "Capacitor_SMD:C_1206_3216Metric"
 			(at 195.2752 48.26 0)
 			(effects

Commit message: workingng on organizing the board
Parts:
- removed C87: 4u7, Capacitor_SMD:C_0603_1608Metric, symbol Device:C
- removed R48, R49: 5k1, Resistor_SMD:R_0402_1005Metric, symbol Device:R
- removed U3: TPD2EUSB30, Package_TO_SOT_SMD:Texas_DRT-3, symbol Power_Protection:TPD2EUSB30
- added C125: 4u7, Capacitor_SMD:C_0603_1608Metric, symbol Device:C
- added R63, R64: 5k1, Resistor_SMD:R_0402_1005Metric, symbol Device:R
- added U13: TPD2EUSB30, Package_TO_SOT_SMD:Texas_DRT-3, symbol Power_Protection:TPD2EUSB30
Connections:
- net +VBUS: now also C125.1
- net GND: now also C125.2, R63.2, R64.2, U13.3 (GND)
- net USB_DM: now also U13.2 (D-)
- net USB_DP: now also U13.1 (D+)
- net at J4.B5 (CC2): now also R64.1
- net at J4.A5 (CC1): now also R63.1
Other:
- moved on the sheet: C100, C101, C102, C103, C104, C105, C106, C107, C108, C109, C124, C88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

Commit message: cleaned up the schematic to look cooler
Parts:
- removed C124, C125, C91: 4u7, Capacitor_SMD:C_0603_1608Metric, symbol Device:C
- removed C88, C90: 470n, Capacitor_SMD:C_0201_0603Metric, symbol Device:C
- removed C89: 47n, Capacitor_SMD:C_0603_1608Metric, symbol Device:C
- removed C92: 47u, Capacitor_SMD:C_1206_3216Metric, symbol Device:C
- removed J4: TYPE-C-31-M-12, Connector_USB:USB_C_Receptacle_HRO_TYPE-C-31-M-12, symbol Connector:USB_C_Receptacle_USB2.0_16P
- removed L5: 1u5, Inductor_SMD:L_Sunlord_SWPA4030S, symbol Device:L
- removed R50: 100k, Resistor_SMD:R_0402_1005Metric, symbol Device:R
- removed R63, R64: 5k1, Resistor_SMD:R_0402_1005Metric, symbol Device:R
- removed U13: TPD2EUSB30, Package_TO_SOT_SMD:Texas_DRT-3, symbol Power_Protection:TPD2EUSB30
- removed U8: TPS62132, Package_DFN_QFN:VQFN-16-1EP_3x3mm_P0.5mm_EP1.68x1.68mm_ThermalVias, symbol Regulator_Switching:TPS62132
Connections:
- no-connect marks 28 -> 26
Other:
- note removed: "1.5uH & 47uF for BOM optimization"
- note removed: "23.5ms start up, reduce inrush >"
- moved on the sheet: C100, C101, C102, C103, C104, C105, C106, C107, C108, C109, C93, C94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
