File: PCB/usb.kicad_sch (KiCad schematic)
At the start: 39 parts, among them J2 Conn_ARM_SWD_TagConnect_TC2030, U10 FT2232HQ, U4 TPD2EUSB30, U6 TPD2EUSB30, U9 M93C56-WMN6TP, Y2 12MHz

Commit message: cleaning up the ft2232H decoupling, laying it out on the PCB too
Parts:
- C101, C103: value 470n -> 4u7; footprint Capacitor_SMD:C_0201_0603Metric -> Capacitor_SMD:C_0603_1608Metric
Other:
- note removed: "^ VCORE ^"
Changed lines of the file:
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@@
 		)
 	)
-	(text "^ VCORE ^"
-		(exclude_from_sim no)
-		(at 140.97 140.716 0)
-		(effects
-			(font
-				(size 1.016 1.016)
-			)
-		)
-	)
 	(junction
 		(at 102.87 194.31)
@@
 			)
 		)
-		(property "Value" "470n"
+		(property "Value" "4u7"
 			(at 141.986 93.218 0)
 			(effects
@@
 			)
 		)
-		(property "Footprint" "Capacitor_SMD:C_0201_0603Metric"
+		(property "Footprint" "Capacitor_SMD:C_0603_1608Metric"
 			(at 141.9352 93.98 0)
 			(effects
@@
 			)
 		)
-		(property "Value" "470n"
+		(property "Value" "4u7"
 			(at 150.876 69.088 0)
 			(effects
@@
 			)
 		)
-		(property "Footprint" "Capacitor_SMD:C_0201_0603Metric"
+		(property "Footprint" "Capacitor_SMD:C_0603_1608Metric"
 			(at 150.8252 69.85 0)
 			(effects

Commit message: working on routing USB and JTAG
Connections:
- net USB_DM renamed USB_D-
- net USB_DP renamed USB_D+
