File: PCB/PCB.kicad_pcb (KiCad board)
At the start: 6 copper layers, 22 x 80 mm, 269 parts, among them J1 Bus_M.2_Edge_M, J2 Conn_ARM_SWD_TagConnect_TC2030, J4 TYPE-C-31-M-12, J7 HDMI_D_1.4, SW1 SW_Push, U1 XC7A50T-FGG484, U10 FT2232HQ, U11 MT41J128M16JT-125:K, U12 PCA9306DC1, U14 UCL0524P, U15 UCL0524P, U16 UCL0524P, U17 TPS62132, U2 MAX20029ATIA/V+, U3 TPD2EUSB30, U4 TPD2EUSB30, U5 TPS2121RUXR, U6 TPD2EUSB30, U7 MT25QL128ABA1EW7-0SIT, U9 M93C56-WMN6TP, Y2 12MHz, Y3 100MHz

Commit message: routing aa bunch of grounds for simple routing
Routing:
- net GND: track 107.2 -> 116.7 mm, vias 82 -> 94
Changed lines of the file:
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@@
+	)
+	(segment
+		(start 152.25 108)
+		(end 151.75 107.5)
+		(width 0.5)
+		(layer "F.Cu")
+		(net 1)
+	)
+	(segment
+		(start 149.25 96)
+		(end 148.25 97)
+		(width 0.5)
+		(layer "F.Cu")
+		(net 1)
 	)
 	(segment
@@
 	)
 	(segment
+		(start 134.25 101)
+		(end 134.75 101.5)
+		(width 0.5)
+		(layer "F.Cu")
+		(net 1)
+	)
+	(segment
 		(start 134.25 91)
 		(end 134.7 91.45)
@@
 	)
 	(segment
+		(start 136.25 87)
+		(end 136.75 87.5)
+		(width 0.5)
+		(layer "F.Cu")
+		(net 1)
+	)
+	(segment
 		(start 146.25 101)
 		(end 145.25 102)
@@
 	)
 	(segment
+		(start 152.25 106)
+		(end 151.75 106.5)
+		(width 0.5)
+		(layer "F.Cu")
+		(net 1)
+	)
+	(segment
 		(start 144.25 93)
 		(end 143.75 93.5)
@@
 	)
 	(segment
+		(start 150.25 99)
+		(end 149.75 99.5)
+		(width 0.5)
+		(layer "F.Cu")
+		(net 1)
+	)
+	(segment
 		(start 146.25 98)
 		(end 146.25 98.088545)
@@
 	)
 	(segment
+		(start 152.25 105)
+		(end 151.75 105.5)
+		(width 0.5)
+		(layer "F.Cu")
+		(net 1)
+	)
+	(segment
 		(start 148.25 95)
 		(end 147.25 96)
@@
 	)
 	(segment
+		(start 146.25 87)
+		(end 145.75 87.5)
+		(width 0.5)
+		(layer "F.Cu")
+		(net 1)
+	)
+	(segment
 		(start 144.25 96.975)
 		(end 143.775 96.5)
@@
 	)
 	(segment
+		(start 133.25 108)
+		(end 133.7 108.45)
+		(width 0.5)
+		(layer "F.Cu")
+		(net 1)
+	)
+	(segment
+		(start 133.25 88)
+		(end 133.75 88.5)
+		(width 0.5)
+		(layer "F.Cu")
+		(net 1)
+	)
+	(segment
 		(start 152.25 95)
 		(end 152.75 95.5)
@@
 	)
 	(segment
+		(start 149.25 96)
+		(end 148.975 96.275)
+		(width 0.5)
+		(layer "F.Cu")
+		(net 1)
+	)
+	(segment
 		(start 143.25 94)
 		(end 143.75 93.5)
@@
 	)
 	(segment
+		(start 133.25 98)
+		(end 133.75 98.5)
+		(width 0.5)
+		(layer "F.Cu")
+		(net 1)
+	)
+	(segment
+		(start 153.25 108)
+		(end 152.75 107.5)
+		(width 0.5)
+		(layer "F.Cu")
+		(net 1)
+	)
+	(segment
 		(start 153.25 98)
 		(end 152.75 97.5)
@@
 	)
 	(via
+		(at 149.75 99.5)
+		(size 0.6)
+		(drill 0.3)
+		(layers "F.Cu" "B.Cu")
+		(net 1)
+	)
+	(via
 		(at 138.35 66.65)
 		(size 0.6)
@@
 	)
 	(via
+		(at 133.75 98.5)
+		(size 0.6)
+		(drill 0.3)
+		(layers "F.Cu" "B.Cu")
+		(net 1)
+	)
+	(via
 		(at 143.75 95.5)
 		(size 0.6)
@@
 	)
 	(via
+		(at 151.75 107.5)
+		(size 0.6)
+		(drill 0.3)
+		(layers "F.Cu" "B.Cu")
+		(net 1)
+	)
+	(via
 		(at 144.75 98.5)
 		(size 0.6)
@@
 	)
 	(via
+		(at 145.75 87.5)
+		(size 0.6)
+		(drill 0.3)
+		(layers "F.Cu" "B.Cu")
+		(net 1)
+	)
+	(via
 		(at 142.75 102.5)
 		(size 0.6)
@@
 	)
 	(via
+		(at 151.75 105.5)
+		(size 0.6)
+		(drill 0.3)
+		(layers "F.Cu" "B.Cu")
+		(net 1)
+	)
+	(via
 		(at 142.75 87.5)
 		(size 0.6)
@@
 	)
 	(via
+		(at 151.75 106.5)
+		(size 0.6)
+		(drill 0.3)
+		(layers "F.Cu" "B.Cu")
+		(net 1)
+	)
+	(via
+		(at 152.75 107.5)
+		(size 0.6)
+		(drill 0.3)
+		(layers "F.Cu" "B.Cu")
+		(net 1)
+	)
+	(via
 		(at 147.75 93.5)
 		(size 0.6)
@@
 	)
 	(via
+		(at 148.775 96.475)
+		(size 0.6)
+		(drill 0.3)
+		(layers "F.Cu" "B.Cu")
+		(net 1)
+	)
+	(via
 		(at 135.75 96.5)
 		(size 0.6)
@@
 	)
 	(via
+		(at 133.7 108.45)
+		(size 0.6)
+		(drill 0.3)
+		(layers "F.Cu" "B.Cu")
+		(net 1)
+	)
+	(via
 		(at 147.7625 99.4875)
 		(size 0.6)
@@
 	)
 	(via
+		(at 134.75 101.5)
+		(size 0.6)
+		(drill 0.3)
+		(layers "F.Cu" "B.Cu")
+		(net 1)
+	)
+	(via
 		(at 136.75 89.5)
 		(size 0.6)
@@
 	)
 	(via
+		(at 136.75 87.5)
+		(size 0.6)
+		(drill 0.3)
+		(layers "F.Cu" "B.Cu")
+		(net 1)
+	)
+	(via
 		(at 153.75 90.5)
 		(size 0.6)
@@
 		(size 0.6)
 		(drill 0.3)
+		(layers "F.Cu" "B.Cu")
+		(net 1)
+	)
+	(via
+		(at 133.75 88.5)
+		(size 0.6)
+		(drill 0.3)

Commit message: faning out GTP decoupling
Routing:
- net GND: track 116.7 -> 127.3 mm, vias 94 -> 109
- net +1V2: track 0.00 -> 4.95 mm, vias 0 -> 4

Commit message: finished decoupling the GTP transceivers!
Parts:
- C35, C36, C37, C38, C39, C40: moved to B.Cu
- moved C37 44.1 mm to (148.8, 105.0), turned to -90 degrees
- moved C40 42.3 mm to (146.7, 108.0), turned to -90 degrees
- moved C39 24.8 mm to (151.5, 107.0), turned to -90 degrees
- moved C35 24.2 mm to (150.5, 104.0), turned to 90 degrees
- moved C36 19.5 mm to (146.3, 103.2), turned to 180 degrees
- moved C38 16.9 mm to (143.1, 107.0), turned to 90 degrees
- moved C169 2.64 mm to (139.8, 105.8), turned to 180 degrees
Routing:
- net Net-(C35-Pad1): track 0.00 -> 8.00 mm, vias 0 -> 5
- net GND: track 127.3 -> 131.7 mm, vias 109 -> 106
- net +1V2: track 4.95 -> 7.61 mm

Commit message: cleaning up silkscreen and some routing
Routing:
- net +1V2: track 7.61 -> 8.39 mm, vias 4 -> 5
Changed lines of the file:
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@@
 			(at 0 1.05 0)
 			(layer "B.SilkS")
+			(hide yes)
 			(effects
 				(font
@@
 			(at 0 1.05 90)
 			(layer "B.SilkS")
+			(hide yes)
 			(effects
 				(font
@@
 			(at 0 1.43 90)
 			(layer "B.SilkS")
+			(hide yes)
 			(effects
 				(font
@@
 			(at 0 1.05 90)
 			(layer "B.SilkS")
+			(hide yes)
 			(effects
 				(font
@@
 			(at 0 1.43 90)
 			(layer "B.SilkS")
+			(hide yes)
 			(effects
 				(font
@@
 			(at 0 1.05 90)
 			(layer "B.SilkS")
+			(hide yes)
 			(effects
 				(font
@@
 	)
 	(segment
-		(start 146.25 107)
-		(end 145.75 107.5)
+		(start 145.75 107.5)
+		(end 146.25 107)
 		(width 0.5)
 		(layer "F.Cu")
@@
 		(net 19)
 	)
+	(via
+		(at 146.7625 106.4875)
+		(size 0.6)
+		(drill 0.3)
+		(layers "F.Cu" "B.Cu")
+		(net 19)
+	)
 	(segment
 		(start 150.98 106.68)
@@
 	)
 	(segment
+		(start 146.7625 107.2125)
+		(end 146.725 107.25)
+		(width 0.5)
+		(layer "B.Cu")
+		(net 19)
+	)
+	(segment
 		(start 143.57 107.32)
 		(end 143.75 107.5)
@@
 		(width 0.5)
 		(layer "B.Cu")
+		(net 19)
+	)
+	(segment
+		(start 146.7625 106.4875)
+		(end 146.7625 107.2125)
+		(width 0.5)
+		(layer "B.Cu")

Commit message: getting ready for DDR routing
Parts:
- moved R55 0.38 mm to (143.9, 69.2)
- moved U3 0.38 mm to (144.8, 67.8)
- moved C101 0.33 mm to (143.8, 71.3)
- moved U11 0.26 mm to (147.5, 77.9)
- moved J2 0.22 mm to (150.8, 67.4)
- moved J4 0.22 mm to (150.8, 67.4)
Changed lines of the file:
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@@
 	(footprint "Package_TO_SOT_SMD:Texas_DRT-3"
 		(layer "F.Cu")
-		(at 144.75 68.225 -90)
+		(at 144.75 67.85 -90)
 		(descr "Texas Instrument DRT-3 1x0.8mm Pitch 0.7mm http://www.ti.com/lit/ds/symlink/tpd2eusb30.pdf")
 		(tags "DRT-3 1x0.8mm Pitch 0.7mm")
@@
 	(footprint "Resistor_SMD:R_0402_1005Metric"
 		(layer "F.Cu")
-		(at 143.95 69.6 180)
+		(at 143.95 69.225 180)
 		(descr "Resistor SMD 0402 (1005 Metric), square (rectangular) end terminal, IPC-7351 nominal, (Body size source: IPC-SM-782 page 72, https://www.pcb-3d.com/wordpress/wp-content/uploads/ipc-sm-782a_amendment_1_and_2.pdf), generated with kicad-footprint-generator")
 		(tags "resistor")
@@
 	(footprint "Capacitor_SMD:C_0603_1608Metric"
 		(layer "F.Cu")
-		(at 143.75 71.6 -90)
+		(at 143.75 71.27 -90)
 		(descr "Capacitor SMD 0603 (1608 Metric), square (rectangular) end terminal, IPC-7351 nominal, (Body size source: IPC-SM-782 page 76, https://www.pcb-3d.com/wordpress/wp-content/uploads/ipc-sm-782a_amendment_1_and_2.pdf), generated with kicad-footprint-generator")
 		(tags "capacitor")
@@
 	(footprint "Package_BGA:Micron_FBGA-96_8x14mm_Layout9x16_P0.8mm"
 		(layer "F.Cu")
-		(at 147.6 78.1 90)
+		(at 147.475 77.875 90)
 		(descr "FBGA-96, 8.0x14.0mm, 96 Ball, 9x16 Layout, 0.8mm Pitch, generated with kicad-footprint-generator ipc_bga_generator.py, https://www.micron.com/-/media/client/global/documents/products/data-sheet/dram/ddr3/4gb_ddr3l.pdf#page=28")
 		(tags "BGA 96 0.8 DDR3 DDR3L DDR4")
@@
 	(footprint "Connector_USB:USB_C_Receptacle_HRO_TYPE-C-31-M-12"
 		(layer "F.Cu")
-		(at 150.815 67.65 90)
+		(at 150.82 67.43 90)
 		(descr "USB Type-C receptacle for USB 2.0 and PD, http://www.krhro.com/uploads/soft/180320/1-1P320120243.pdf")
 		(tags "usb usb-c 2.0 pd")
@@
 	(footprint "Connector:Tag-Connect_TC2030-IDC-FP_2x03_P1.27mm_Vertical"
 		(layer "B.Cu")
-		(at 150.84 67.65 180)
+		(at 150.845 67.43 180)
 		(descr "Tag-Connect programming header; http://www.tag-connect.com/Materials/TC2030-IDC.pdf")
 		(tags "tag connect programming header pogo pins")
@@
 			(polygon
 				(pts
-					(xy 149.57 67.015) (xy 152.11 67.015) (xy 152.11 68.285) (xy 149.57 68.285)
+					(xy 149.575 66.795) (xy 152.115 66.795) (xy 152.115 68.065) (xy 149.575 68.065)
 				)
 			)

Commit message: did the DDR3 decoupling fanout
Routing:
- net GND: track 131.7 -> 141.6 mm, vias 106 -> 127
- net +1V5: track 19.3 -> 27.0 mm, vias 12 -> 30

Commit message: routed DDR3 VDD
Parts:
- C59, C60, C61, C62, C63, C64, C65, C73, C74: moved to B.Cu
- moved C62 49.9 mm to (152.8, 82.1)
- moved C63 49.0 mm to (148.0, 81.3), turned to 180 degrees
- moved C74 48.3 mm to (144.3, 74.8), turned to -90 degrees
- moved C59 46.0 mm to (150.4, 82.1), turned to 180 degrees
- moved C61 44.7 mm to (141.2, 80.2), turned to 90 degrees
- moved C73 40.0 mm to (145.8, 75.6), turned to 90 degrees
- moved C60 39.4 mm to (148.0, 75.9), turned to 180 degrees
- moved C64 39.3 mm to (150.4, 73.6), turned to 180 degrees
- moved C65 36.5 mm to (152.8, 73.6)
Routing:
- net GND: track 141.6 -> 148.5 mm
- net +1V5: track 27.0 -> 33.8 mm

Commit message: finished decoupling my DDR3!
Parts:
- C76, C77, C78, C79, C80, C81, C82, C83, C84: moved to B.Cu
- moved C76 54.3 mm to (141.6, 82.1)
- moved C81 52.6 mm to (144.0, 79.8)
- moved C80 52.3 mm to (140.5, 74.8), turned to 90 degrees
- moved C77 51.6 mm to (143.4, 82.1)
- moved C82 50.6 mm to (146.1, 80.7), turned to -90 degrees
- moved C78 48.9 mm to (145.3, 82.1), turned to 180 degrees
- moved C83 46.9 mm to (142.4, 75.1), turned to 180 degrees
- moved C84 40.9 mm to (147.6, 73.7), turned to 180 degrees
- moved C79 40.3 mm to (145.7, 73.7)
- moved C126 0.07 mm to (138.6, 73.9)
- moved C106 0.06 mm to (137.8, 72.8)
Routing:
- net +1V5: track 33.8 -> 41.2 mm
- net GND: track 148.5 -> 155.8 mm
