File: PCB/PCB.kicad_pcb (KiCad board)
At the start: 6 copper layers, 22 x 80 mm, 270 parts, among them J1 Bus_M.2_Edge_M, J2 Conn_ARM_SWD_TagConnect_TC2030, J4 TYPE-C-31-M-12, J7 HDMI_D_1.4, SW1 SW_Push, U1 XC7A50T-FGG484, U10 FT2232HQ, U11 MT41J128M16JT-125:K, U12 PCA9306DC1, U14 UCL0524P, U15 UCL0524P, U16 UCL0524P, U17 TPS62132, U2 MAX20029ATIA/V+, U3 TPD2EUSB30, U4 TPD2EUSB30, U5 TPS2121RUXR, U6 TPD2EUSB30, U7 MT25QL128ABA1EW7-0SIT, U9 M93C56-WMN6TP, Y2 12MHz, Y3 100MHz

Commit message: DDR signal fanout
Parts:
- moved C82 0.13 mm to (145.6, 80.7)
Routing:
- net /Artix 7 Banks/DDR_DQ14: track 0.00 -> 0.42 mm, vias 0 -> 1
- net Net-(U11A-ZQ): track 0.00 -> 0.42 mm, vias 0 -> 1
- net /Artix 7 Banks/DDR_DQ3: track 0.00 -> 0.42 mm, vias 0 -> 1
- net /Artix 7 Banks/DDR_BA1: track 0.00 -> 0.42 mm, vias 0 -> 1
- net /Artix 7 Banks/DDR_DQ6: track 0.00 -> 0.42 mm, vias 0 -> 1
- net /Artix 7 Banks/DDR_DQ2: track 0.00 -> 0.42 mm, vias 0 -> 1
- net /Artix 7 Banks/DDR_A6: track 0.00 -> 0.42 mm, vias 0 -> 1
- net /Artix 7 Banks/DDR_DQ5: track 0.00 -> 0.42 mm, vias 0 -> 1
- net /Artix 7 Banks/DDR_DQ11: track 0.00 -> 0.42 mm, vias 0 -> 1
- net Net-(U11A-~{CS}): track 0.00 -> 0.41 mm, vias 0 -> 1
- net /Artix 7 Banks/DDR_A3: track 0.00 -> 0.41 mm, vias 0 -> 1
- net /Artix 7 Banks/DDR_A4: track 0.00 -> 0.41 mm, vias 0 -> 1
- net /Artix 7 Banks/DDR_DQ10: track 0.00 -> 0.41 mm, vias 0 -> 1
- net /Artix 7 Banks/DDR_BA0: track 0.00 -> 0.41 mm, vias 0 -> 1
- net /Artix 7 Banks/DDR_A5: track 0.00 -> 0.41 mm, vias 0 -> 1
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
Commit message: working on DDR3 routing, this is going to be rough...
Parts:
- moved C127 0.50 mm to (137.6, 76.3)
- moved C129 0.50 mm to (137.6, 77.8)
- moved C131 0.50 mm to (136.3, 84.5)
- moved U17 0.50 mm to (135.0, 76.4)
- moved R65 0.50 mm to (133.3, 79.2)
- moved C130 0.50 mm to (138.7, 77.2)
- moved L6 0.50 mm to (136.2, 80.9)
- turned Y3 to 180 degrees
Routing:
- net /Artix 7 Banks/DDR_DQ1: track 0.00 -> 11.4 mm
- net /Artix 7 Banks/DDR_DQM0: track 0.00 -> 11.0 mm
- net /Artix 7 Banks/DDR_DQ8: track 0.00 -> 10.8 mm
- net /Artix 7 Banks/DDR_DQS1+: track 0.00 -> 10.6 mm
- net /Artix 7 Banks/DDR_DQS1-: track 0.00 -> 10.3 mm
- net /Artix 7 Banks/DDR_DQ12: track 0.00 -> 9.77 mm
- net /Artix 7 Banks/DDR_A8: track 0.00 -> 9.71 mm
- net /Artix 7 Banks/DDR_A11: track 0.00 -> 8.77 mm
- net /Artix 7 Banks/DDR_A14: track 0.00 -> 8.67 mm

Commit message: DDR command netclasses and some more routing
Parts:
- R23: moved to B.Cu
- moved R23 44.2 mm to (148.3, 82.6), turned to -90 degrees
- moved R16 16.3 mm to (162.9, 51.1), turned to 180 degrees
Routing:
- net /Artix 7 Banks/~{DDR_ODT}: track 0.00 -> 1.25 mm, vias 0 -> 1
- net GND: track 159.7 -> 160.1 mm, vias 132 -> 133

Commit message: faning out more DDR3, crosstalk looking BAD
Parts:
- moved R65 1.78 mm to (131.6, 79.2), turned to -90 degrees
- moved L6 1.11 mm to (135.1, 80.9)
- moved C131 1.11 mm to (135.2, 84.4)
- moved C130 0.95 mm to (138.7, 76.2)
- moved C59 0.47 mm to (150.5, 82.1), turned to 0 degrees
Routing:
- net /Artix 7 Banks/DDR_DQ5: track 0.42 -> 14.2 mm
- net /Artix 7 Banks/DDR_DQ3: track 0.42 -> 12.7 mm
- net /Artix 7 Banks/DDR_DQ10: track 0.41 -> 11.0 mm
- net /Artix 7 Banks/DDR_DQ14: track 0.42 -> 10.9 mm
- net /Artix 7 Banks/DDR_A3: track 0.41 -> 9.45 mm
- net /Artix 7 Banks/DDR_DQ11: track 0.42 -> 9.07 mm
- net /Artix 7 Banks/DDR_A5: track 0.41 -> 7.72 mm
- net /Artix 7 Banks/DDR_DQ15: track 0.00 -> 5.51 mm, vias 0 -> 1
- net /Artix 7 Banks/DDR_A7: track 0.41 -> 5.82 mm
- net /Artix 7 Banks/DDR_DQ13: track 0.00 -> 4.71 mm
- net /Artix 7 Banks/DDR_BA0: track 0.41 -> 4.58 mm
- net Net-(U11A-~{CS}): track 0.41 -> 4.54 mm
- net /Artix 7 Banks/DDR_DQ7: track 0.00 -> 0.42 mm, vias 0 -> 1

Commit message: minimizing crosstalk and adding in CLK net class
Routing:
- net /Artix 7 Banks/DDR_A3: track 9.45 -> 10.1 mm
- net /Artix 7 Banks/DDR_A7: track 5.82 -> 6.34 mm
- net /Artix 7 Banks/DDR_A5: track 7.72 -> 8.23 mm
- net /Artix 7 Banks/~{DDR_RESET}: track 0.00 -> 0.42 mm, vias 0 -> 1
Changed lines of the file:
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@@
+	)
+	(segment
+		(start 153.1 80.25)
+		(end 152.805418 80.544584)
+		(width 0.1862)
+		(layer "F.Cu")
+		(net 334)
+	)
+	(via
+		(at 152.805418 80.544584)
+		(size 0.45)
+		(drill 0.2)
+		(layers "F.Cu" "B.Cu")
+		(net 334)
 	)
 	(segment
@@
 	)
 	(segment
-		(start 142.425 77.325)
-		(end 141.525 77.325)
+		(start 143.5 76.25)
+		(end 142.4 77.35)
 		(width 0.1862)
 		(layer "F.Cu")
@@
 	)
 	(segment
-		(start 141.525 77.325)
-		(end 138.875 79.975)
+		(start 142.4 77.35)
+		(end 141.05 77.35)
 		(width 0.1862)
 		(layer "F.Cu")
@@
 	)
 	(segment
-		(start 138.875 79.975)
+		(start 138.875 79.525)
 		(end 138.875 84.6)
 		(width 0.1862)
@@
 	)
 	(segment
-		(start 143.5 76.25)
-		(end 142.425 77.325)
+		(start 141.05 77.35)
+		(end 138.875 79.525)
 		(width 0.1862)
 		(layer "F.Cu")
@@
 	)
 	(segment
+		(start 141.23 77.8)
+		(end 139.35 79.68)
+		(width 0.1862)
+		(layer "F.Cu")
+		(net 407)
+	)
+	(segment
+		(start 142.75 77.8)
+		(end 141.23 77.8)
+		(width 0.1862)
+		(layer "F.Cu")
+		(net 407)
+	)
+	(segment
+		(start 139.35 79.68)
+		(end 139.35 84.575)
+		(width 0.1862)
+		(layer "F.Cu")
+		(net 407)
+	)
+	(segment
 		(start 144.3 76.25)
-		(end 142.775 77.775)
-		(width 0.1862)
-		(layer "F.Cu")
-		(net 407)
-	)
-	(segment
-		(start 142.075 77.775)
-		(end 141.675 77.775)
-		(width 0.1862)
-		(layer "F.Cu")
-		(net 407)
-	)
-	(segment
-		(start 139.35 80.1)
-		(end 139.35 84.575)
-		(width 0.1862)
-		(layer "F.Cu")
-		(net 407)
-	)
-	(segment
-		(start 141.675 77.775)
-		(end 139.35 80.1)
-		(width 0.1862)
-		(layer "F.Cu")
-		(net 407)
-	)
-	(segment
-		(start 142.775 77.775)
-		(end 142.075 77.775)
+		(end 142.75 77.8)
 		(width 0.1862)
 		(layer "F.Cu")
@@
 	)
 	(segment
+		(start 137.9591 78.6309)
+		(end 137.9591 84.7159)
+		(width 0.1862)
+		(layer "F.Cu")
+		(net 411)
+	)
+	(segment
+		(start 140.34 76.25)
+		(end 137.9591 78.6309)
+		(width 0.1862)
+		(layer "F.Cu")
+		(net 411)
+	)
+	(segment
 		(start 141.1 76.25)
-		(end 137.9591 79.3909)
-		(width 0.1862)
-		(layer "F.Cu")
-		(net 411)
-	)
-	(segment
-		(start 137.9591 79.3909)
-		(end 137.9591 84.7159)
+		(end 140.34 76.25)
 		(width 0.1862)
 		(layer "F.Cu")
@@
 	)
 	(segment
-		(start 153.975 80.575)
+		(start 153.37 79.36)
+		(end 153.975 79.965)
+		(width 0.1862)
+		(layer "B.Cu")
+		(net 413)
+	)
+	(segment
+		(start 153.975 79.965)
 		(end 153.975 84.525)
 		(width 0.1862)
@@
 	)
 	(segment
-		(start 152.944096 79.544096)
-		(end 153.575 80.175)
+		(start 151.21 79.96)
+		(end 151.81 79.36)
 		(width 0.1862)
 		(layer "B.Cu")
@@
 	)
 	(segment
-		(start 153.575 80.175)
-		(end 153.975 80.575)
+		(start 151.81 79.36)
+		(end 153.37 79.36)
 		(width 0.1862)
 		(layer "B.Cu")
@@
 	)
 	(segment
-		(start 151.21 79.96)
-		(end 151.625904 79.544096)
-		(width 0.1862)
-		(layer "B.Cu")
-		(net 413)
-	)
-	(segment
-		(start 151.625904 79.544096)
-		(end 152.944096 79.544096)
-		(width 0.1862)
-		(layer "B.Cu")
-		(net 413)
-	)
-	(segment
-		(start 142.175 78.225)
-		(end 141.682805 78.225)
+		(start 141.39 78.33)
+		(end 139.9 79.82)
 		(width 0.1862)
 		(layer "F.Cu")
@@
 	)
 	(segment
-		(start 143.125 78.225)
-		(end 142.175 78.225)
+		(start 143.02 78.33)
+		(end 141.39 78.33)
 		(width 0.1862)
 		(layer "F.Cu")
@@
 	)
 	(segment
-		(start 141.682805 78.225)
-		(end 139.9 80.007805)
+		(start 145.1 76.25)
+		(end 143.02 78.33)
 		(width 0.1862)
 		(layer "F.Cu")
@@
 	)
 	(segment
-		(start 139.9 80.007805)
+		(start 139.9 79.82)
 		(end 139.9 84.65)
-		(width 0.1862)
-		(layer "F.Cu")
-		(net 414)
-	)
-	(segment
-		(start 145.1 76.25)
-		(end 143.125 78.225)
 		(width 0.1862)
 		(layer "F.Cu")
@@
 	)
 	(segment
+		(start 151.415855 78.95)
+		(end 153.71 78.95)
+		(width 0.1862)
+		(layer "B.Cu")
+		(net 421)
+	)
+	(segment
+		(start 154.4559 79.6959)
+		(end 154.4559 84.575)
+		(width 0.1862)
+		(layer "B.Cu")
+		(net 421)
+	)
+	(segment
+		(start 153.71 78.95)
+		(end 154.4559 79.6959)
+		(width 0.1862)
+		(layer "B.Cu")
+		(net 421)
+	)
+	(segment
 		(start 150.408596 79.957259)
-		(end 151.108959 79.256896)
-		(width 0.1862)
-		(layer "B.Cu")
-		(net 421)
-	)
-	(segment
-		(start 151.108959 79.256896)
-		(end 153.406896 79.256896)
-		(width 0.1862)
-		(layer "B.Cu")
-		(net 421)
-	)
-	(segment
-		(start 153.406896 79.256896)
-		(end 153.925 79.775)
-		(width 0.1862)
-		(layer "B.Cu")
-		(net 421)
-	)
-	(segment
-		(start 154.4559 80.3059)
-		(end 154.4559 84.575)
-		(width 0.1862)
-		(layer "B.Cu")
-		(net 421)
-	)
-	(segment
-		(start 153.925 79.775)
-		(end 154.4559 80.3059)
+		(end 151.415855 78.95)
 		(width 0.1862)
 		(layer "B.Cu")
@@
 		(layer "B.Cu")
 		(net 425)
+	)
+	(segment
+		(start 140.602536 76.7588)
+		(end 138.2588 79.102536)
+		(width 0.1074)
+		(layer "F.Cu")
+		(net 426)
+	)
+	(segment
+		(start 141.9 76.25)
+		(end 141.9 76.721336)
+		(width 0.1074)
+		(layer "F.Cu")
+		(net 426)
 	)
 	(segment
@@
 	(segment
 		(start 141.862536 76.7588)
-		(end 141.151868 76.7588)
+		(end 140.602536 76.7588)
 		(width 0.1074)
 		(layer "F.Cu")
@@
 	)
 	(segment
-		(start 141.9 76.25)
-		(end 141.9 76.721336)
-		(width 0.1074)
-		(layer "F.Cu")
-		(net 426)
-	)
-	(segment
-		(start 141.151868 76.7588)
-		(end 138.2588 79.651868)
-		(width 0.1074)
-		(layer "F.Cu")
-		(net 426)
-	)
-	(segment
-		(start 138.2588 79.651868)
+		(start 138.2588 79.102536)
 		(end 138.2588 84.675)
 		(width 0.1074)
@@
 	)
 	(segment
-		(start 152.021678 79.975)
-		(end 152.6 79.975)
+		(start 153 79.77)
+		(end 153.55 80.32)
 		(width 0.1862)
 		(layer "B.Cu")
@@
 	)
 	(segment
-		(start 152.6 79.975)
-		(end 153.55 80.925)
+		(start 153.55 80.32)
+		(end 153.55 84.4)
 		(width 0.1862)
 		(layer "B.Cu")
@@
 	)
 	(segment
-		(start 153.55 80.925)
-		(end 153.55 84.4)
+		(start 152.20307 79.77)
+		(end 153 79.77)
 		(width 0.1862)
 		(layer "B.Cu")
@@
 	(segment
 		(start 152.009874 79.963196)
-		(end 152.021678 79.975)
+		(end 152.20307 79.77)
 		(width 0.1862)
 		(layer "B.Cu")
@@
 	)
 	(segment
-		(start 138.4912 79.748132)
-		(end 138.4912 84.675)
+		(start 140.6988 76.9912)
+		(end 138.4912 79.1988)
 		(width 0.1074)
 		(layer "F.Cu")
@@
 	(segment
 		(start 141.9588 76.9912)
-		(end 141.248132 76.9912)
+		(end 140.6988 76.9912)
 		(width 0.1074)
 		(layer "F.Cu")
@@
 	)
 	(segment
-		(start 141.248132 76.9912)
-		(end 138.4912 79.748132)
+		(start 138.4912 79.1988)
+		(end 138.4912 84.675)
 		(width 0.1074)
 		(layer "F.Cu")

Commit message: faned out all my I/O's
Parts:
- R16: moved to B.Cu
- moved R16 28.6 mm to (149.7, 76.5), turned to -90 degrees
Routing:
- net /Artix 7 Banks/DDR_A13: track 0.00 -> 1.00 mm, vias 0 -> 1
- net /Artix 7 Banks/DDR_A9: track 0.00 -> 0.98 mm, vias 0 -> 1
- net /Artix 7 Banks/DDR_A2: track 0.00 -> 0.98 mm, vias 0 -> 1
- net Net-(U11A-ZQ): track 0.42 -> 1.36 mm
- net /Artix 7 Banks/DDR_CLK-: track 0.00 -> 0.90 mm, vias 0 -> 1
- net /Artix 7 Banks/DDR_CLK+: track 0.00 -> 0.90 mm, vias 0 -> 1
- net /Artix 7 Banks/DDR_DQS0-: track 0.00 -> 0.89 mm, vias 0 -> 1
- net /Artix 7 Banks/DDR_DQS0+: track 0.00 -> 0.89 mm, vias 0 -> 1
- net GND: track 160.1 -> 160.7 mm, vias 133 -> 134
- net /Artix 7 Banks/~{DDR_RAS}: track 0.00 -> 0.47 mm, vias 0 -> 1
- net /Artix 7 Banks/DDR_CKE: track 0.00 -> 0.47 mm, vias 0 -> 1
- net /Artix 7 Banks/DDR_DQ9: track 0.00 -> 0.46 mm, vias 0 -> 1
- net /Artix 7 Banks/DDR_DQM1: track 0.00 -> 0.46 mm, vias 0 -> 1
- net /Artix 7 Banks/~{DDR_WE}: track 0.00 -> 0.46 mm, vias 0 -> 1
- net /Artix 7 Banks/DDR_DQ0: track 0.00 -> 0.44 mm, vias 0 -> 1
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
Commit message: working on routing innner layers
Parts:
- R28: moved to B.Cu
- moved R28 39.5 mm to (151.6, 80.7), turned to 180 degrees
Routing:
- net /Artix 7 Banks/DDR_BA1: track 0.42 -> 11.7 mm
- net /Artix 7 Banks/DDR_A4: track 0.41 -> 11.4 mm
- net /Artix 7 Banks/DDR_A6: track 0.42 -> 11.1 mm
- net /Artix 7 Banks/DDR_A1: track 0.39 -> 9.67 mm
- net /Artix 7 Banks/DDR_A3: track 10.1 -> 3.47 mm
- net /Artix 7 Banks/~{DDR_CAS}: track 0.44 -> 6.08 mm
- net /Artix 7 Banks/DDR_A2: track 0.98 -> 6.23 mm
- net /Artix 7 Banks/DDR_A5: track 8.18 -> 3.47 mm
- net /Artix 7 Banks/~{DDR_WE}: track 0.46 -> 4.57 mm
- net /Artix 7 Banks/DDR_A0: track 0.43 -> 4.40 mm
- net /Artix 7 Banks/DDR_BA2: track 0.43 -> 4.28 mm
- net /Artix 7 Banks/DDR_A9: track 0.98 -> 4.49 mm
- net /Artix 7 Banks/~{DDR_RESET}: track 0.42 -> 3.36 mm
- net /Artix 7 Banks/DDR_A13: track 1.00 -> 3.54 mm
- net /Artix 7 Banks/DDR_A7: track 6.03 -> 3.50 mm
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
Commit message: some beautiful inner layer routing
Parts:
- R31: moved to B.Cu
- moved R31 34.0 mm to (147.9, 77.3)
Routing:
- net /Artix 7 Banks/DDR_CLK-: track 0.90 -> 16.3 mm
- net /Artix 7 Banks/DDR_CLK+: track 0.90 -> 16.0 mm
- net /Artix 7 Banks/DDR_A10: track 0.41 -> 14.7 mm
- net /Artix 7 Banks/DDR_DQ7: track 0.42 -> 13.3 mm
- net /Artix 7 Banks/DDR_DQS0-: track 0.89 -> 10.8 mm
- net /Artix 7 Banks/DDR_DQS0+: track 0.89 -> 9.77 mm
- net /Artix 7 Banks/DDR_A12: track 0.41 -> 8.48 mm
- net /Artix 7 Banks/~{DDR_RAS}: track 0.47 -> 6.06 mm
- net /Artix 7 Banks/DDR_DQ4: track 0.43 -> 5.94 mm
- net /Artix 7 Banks/DDR_DQ9: track 0.46 -> 5.31 mm
- net /Artix 7 Banks/DDR_DQ0: track 0.44 -> 5.27 mm
- net /Artix 7 Banks/DDR_DQM1: track 0.46 -> 5.27 mm
- net /Artix 7 Banks/DDR_DQ6: track 0.42 -> 4.79 mm
- net /Artix 7 Banks/DDR_DQ2: track 0.42 -> 4.65 mm
- net /Artix 7 Banks/~{DDR_CAS}: track 6.08 -> 4.98 mm
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