File: PCB/PCB.kicad_pcb (KiCad board)
At the start: 6 copper layers, 22 x 80 mm, 270 parts, among them J1 Bus_M.2_Edge_M, J2 Conn_ARM_SWD_TagConnect_TC2030, J4 TYPE-C-31-M-12, J7 HDMI_D_1.4, SW1 SW_Push, U1 XC7A50T-FGG484, U10 FT2232HQ, U11 MT41J128M16JT-125:K, U12 PCA9306DC1, U14 UCL0524P, U15 UCL0524P, U16 UCL0524P, U17 TPS62132, U2 MAX20029ATIA/V+, U3 TPD2EUSB30, U4 TPD2EUSB30, U5 TPS2121RUXR, U6 TPD2EUSB30, U7 MT25QL128ABA1EW7-0SIT, U9 M93C56-WMN6TP, Y2 12MHz, Y3 100MHz

Commit message: finished the IO fanout
Parts:
- moved C82 0.55 mm to (145.4, 81.2)
- moved C63 0.15 mm to (146.8, 79.9)

Commit message: modifying DDR3 CS, routing it too
Parts:
- R42: value 100 -> 1k
- moved R42 20.1 mm to (149.5, 78.6), turned to -90 degrees
Routing:
- net Net-(U11A-~{CS}): track 0.00 -> 1.31 mm, vias 0 -> 1
- net GND: track 163.5 -> 164.1 mm, vias 133 -> 134
Changed lines of the file:
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@@
 	(footprint "Resistor_SMD:R_0402_1005Metric"
 		(layer "B.Cu")
-		(at 169.585 78.43 180)
+		(at 149.5 78.6 -90)
 		(descr "Resistor SMD 0402 (1005 Metric), square (rectangular) end terminal, IPC-7351 nominal, (Body size source: IPC-SM-782 page 72, https://www.pcb-3d.com/wordpress/wp-content/uploads/ipc-sm-782a_amendment_1_and_2.pdf), generated with kicad-footprint-generator")
 		(tags "resistor")
 		(property "Reference" "R42"
-			(at 0 1.17 0)
+			(at 0 1.17 90)
 			(layer "B.SilkS")
 			(hide yes)
@@
 			)
 		)
-		(property "Value" "100"
-			(at 0 -1.17 0)
+		(property "Value" "1k"
+			(at 0 -1.17 90)
 			(layer "B.Fab")
 			(effects
@@
 		)
 		(property "Datasheet" "~"
-			(at 0 0 0)
+			(at 0 0 90)
 			(layer "B.Fab")
 			(hide yes)
@@
 		)
 		(property "Description" "Resistor"
-			(at 0 0 0)
+			(at 0 0 90)
 			(layer "B.Fab")
 			(hide yes)
@@
 		)
 		(fp_line
-			(start 0.93 0.47)
-			(end 0.93 -0.47)
+			(start -0.93 0.47)
+			(end 0.93 0.47)
 			(stroke
 				(width 0.05)
@@
 		)
 		(fp_line
-			(start 0.93 -0.47)
-			(end -0.93 -0.47)
+			(start 0.93 0.47)
+			(end 0.93 -0.47)
 			(stroke
 				(width 0.05)
@@
 		)
 		(fp_line
-			(start -0.93 0.47)
-			(end 0.93 0.47)
+			(start -0.93 -0.47)
+			(end -0.93 0.47)
 			(stroke
 				(width 0.05)
@@
 		)
 		(fp_line
-			(start -0.93 -0.47)
-			(end -0.93 0.47)
+			(start 0.93 -0.47)
+			(end -0.93 -0.47)
 			(stroke
 				(width 0.05)
@@
 		)
 		(fp_line
-			(start 0.525 0.27)
-			(end 0.525 -0.27)
+			(start -0.525 0.27)
+			(end 0.525 0.27)
 			(stroke
 				(width 0.1)
@@
 		)
 		(fp_line
-			(start 0.525 -0.27)
-			(end -0.525 -0.27)
+			(start 0.525 0.27)
+			(end 0.525 -0.27)
 			(stroke
 				(width 0.1)
@@
 		)
 		(fp_line
-			(start -0.525 0.27)
-			(end 0.525 0.27)
+			(start -0.525 -0.27)
+			(end -0.525 0.27)
 			(stroke
 				(width 0.1)
@@
 		)
 		(fp_line
-			(start -0.525 -0.27)
-			(end -0.525 0.27)
+			(start 0.525 -0.27)
+			(end -0.525 -0.27)
 			(stroke
 				(width 0.1)
@@
 		)
 		(fp_text user "${REFERENCE}"
-			(at 0 0 0)
+			(at 0 0 90)
 			(layer "B.Fab")
 			(effects
@@
 		)
 		(pad "1" smd roundrect
-			(at -0.51 0 180)
+			(at -0.51 0 270)
 			(size 0.54 0.64)
 			(layers "B.Cu" "B.Mask" "B.Paste")
@@
 		)
 		(pad "2" smd roundrect
-			(at 0.51 0 180)
+			(at 0.51 0 270)
 			(size 0.54 0.64)
 			(layers "B.Cu" "B.Mask" "B.Paste")
@@
 	)
 	(via
+		(at 150.1 78.1)
+		(size 0.45)
+		(drill 0.2)
+		(layers "F.Cu" "B.Cu")
+		(net 1)
+	)
+	(via
 		(at 149.775 102.525)
 		(size 0.6)
@@
 	)
 	(segment
+		(start 150.09 78.09)
+		(end 150.1 78.1)
+		(width 0.2)
+		(layer "B.Cu")
+		(net 1)
+	)
+	(segment
 		(start 145.955 103.2)
 		(end 145.955 102.705)
@@
 	)
 	(segment
+		(start 149.5 78.09)
+		(end 150.09 78.09)
+		(width 0.2)
+		(layer "B.Cu")
+		(net 1)
+	)
+	(segment
 		(start 148.7 81.23)
 		(end 149.28 81.23)
@@
 	)
 	(segment
+		(start 149.1 80.25)
+		(end 149.5 79.85)
+		(width 0.2)
+		(layer "F.Cu")
+		(net 366)
+	)
+	(via
+		(at 149.5 79.85)
+		(size 0.45)
+		(drill 0.2)
+		(layers "F.Cu" "B.Cu")
+		(net 366)
+	)
+	(segment
+		(start 149.5 79.85)
+		(end 149.5 79.11)
+		(width 0.2)
+		(layer "B.Cu")
+		(net 366)
+	)
+	(segment
 		(start 149.9 75.45)
 		(end 149.5 75.05)
@@
 	(segment
 		(start 150.3 79.05)
-		(end 149.05 80.3)
+		(end 149.5 79.05)
+		(width 0.1308)
+		(layer "In2.Cu")
+		(net 417)
+	)
+	(segment
+		(start 149.5 79.05)
+		(end 149.05 79.5)
 		(width 0.1308)
 		(layer "In2.Cu")
@@
 	)
 	(segment
-		(start 149.05 80.3)
-		(end 149.05 82.1)
+		(start 149.05 79.5)
+		(end 149.05 82)
 		(width 0.1308)
 		(layer "In2.Cu")

Commit message: found a couple stray pins not routed, finally did themgit add .
Parts:
- moved R16 21.3 mm to (148.9, 73.6), turned to 90 degrees
- moved R28 13.8 mm to (159.0, 75.9), turned to 90 degrees
- moved R30 13.3 mm to (156.9, 75.9), turned to -90 degrees
- moved C73 0.89 mm to (148.2, 75.1)
- moved C13 0.10 mm to (150.0, 75.8)
Routing:
- net /Artix 7 Banks/DDR_CKE: track 0.00 -> 16.6 mm, vias 0 -> 1
- net /Artix 7 Banks/DDR_DQ5: track 0.57 -> 13.7 mm
- net /Artix 7 Banks/DDR_A12: track 15.7 -> 6.93 mm
- net /Artix 7 Banks/DDR_A10: track 15.6 -> 7.51 mm
- net /Artix 7 Banks/DDR_DQM0: track 16.7 -> 10.9 mm
- net /Artix 7 Banks/~{DDR_ODT}: track 1.40 -> 6.28 mm
- net /Artix 7 Banks/DDR_DQM1: track 8.40 -> 5.46 mm
- net /Artix 7 Banks/DDR_DQ0: track 6.29 -> 3.73 mm
- net /Artix 7 Banks/DDR_DQ8: track 24.5 -> 22.5 mm
- net Net-(U11A-ZQ): track 0.57 -> 2.34 mm
- net /Artix 7 Banks/DDR_DQ6: track 5.30 -> 3.54 mm
- net /Artix 7 Banks/DDR_CLK+: track 16.3 -> 14.7 mm
- net /Artix 7 Banks/DDR_CLK-: track 16.2 -> 14.7 mm
- net /Artix 7 Banks/DDR_DQ7: track 12.8 -> 11.8 mm
- net /Artix 7 Banks/DDR_DQ1: track 12.4 -> 11.4 mm
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
Commit message: finished my DDR fanout after adding the pulldowns
Parts:
- R28: moved to F.Cu
- moved R30 12.2 mm to (144.7, 77.0), turned to 90 degrees
- moved R28 10.5 mm to (151.6, 83.4), turned to 180 degrees
Routing:
- net /Artix 7 Banks/~{DDR_RESET}: track 2.41 -> 3.89 mm
- net GND: track 163.9 -> 165.3 mm, vias 135 -> 137

Commit message: hopping off for the night, looking sick!
Routing:
- net /Artix 7 Banks/DDR_DQ13: track 3.82 -> 10.3 mm
- net /Artix 7 Banks/~{DDR_WE}: track 2.67 -> 7.71 mm
- net /Artix 7 Banks/DDR_DQ2: track 3.02 -> 7.48 mm
- net /Artix 7 Banks/~{DDR_ODT}: track 6.28 -> 9.63 mm
- net /Artix 7 Banks/DDR_A13: track 4.32 -> 7.62 mm
- net /Artix 7 Banks/~{DDR_RESET}: track 3.89 -> 6.89 mm
- net /Artix 7 Banks/DDR_A14: track 8.27 -> 10.6 mm
- net /Artix 7 Banks/DDR_DQ15: track 4.79 -> 3.18 mm
Changed lines of the file:
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@@
+	)
+	(segment
+		(start 147.9 81.85)
+		(end 147.2 82.55)
+		(width 0.1862)
+		(layer "F.Cu")
+		(net 316)
+	)
+	(segment
+		(start 147.2 83.9)
+		(end 149.25 85.95)
+		(width 0.1862)
+		(layer "F.Cu")
+		(net 316)
 	)
 	(segment
@@
 	)
 	(segment
-		(start 147.6 82.15)
-		(end 147.2 82.55)
+		(start 149.25 86.25)
+		(end 149.25 86.5)
 		(width 0.1862)
 		(layer "F.Cu")
@@
 	(segment
 		(start 147.2 82.55)
-		(end 147.2 84)
+		(end 147.2 83.9)
 		(width 0.1862)
 		(layer "F.Cu")
@@
 	)
 	(segment
-		(start 147.9 81.85)
-		(end 147.6 82.15)
+		(start 149.25 85.95)
+		(end 149.25 86.25)
 		(width 0.1862)
 		(layer "F.Cu")
@@
 	)
 	(segment
+		(start 152.25 83.54)
+		(end 152.25 86.35)
+		(width 0.1862)
+		(layer "F.Cu")
+		(net 334)
+	)
+	(segment
 		(start 153.494101 80.644101)
 		(end 153.494101 81.655899)
@@
 		(start 153.1 80.25)
 		(end 153.494101 80.644101)
+		(width 0.1862)
+		(layer "F.Cu")
+		(net 334)
+	)
+	(segment
+		(start 152.11 83.4)
+		(end 152.25 83.54)
 		(width 0.1862)
 		(layer "F.Cu")
@@
 	)
 	(segment
+		(start 148.7 81.725)
+		(end 150.25 83.275)
+		(width 0.1862)
+		(layer "F.Cu")
+		(net 397)
+	)
+	(segment
+		(start 148.7 79.85)
+		(end 148.7 81.725)
+		(width 0.1862)
+		(layer "F.Cu")
+		(net 397)
+	)
+	(segment
 		(start 149.1 79.45)
 		(end 148.7 79.85)
@@
 	)
 	(segment
-		(start 148.7 79.85)
-		(end 148.7 81.95)
+		(start 150.25 83.275)
+		(end 150.25 86.35)
 		(width 0.1862)
 		(layer "F.Cu")
@@
 	)
 	(segment
+		(start 148.2 86)
+		(end 148.2 86.45)
+		(width 0.1862)
+		(layer "F.Cu")
+		(net 399)
+	)
+	(segment
 		(start 145.1 80.25)
 		(end 145.5 80.65)
@@
 	)
 	(segment
+		(start 146.45 84.25)
+		(end 148.1 85.9)
+		(width 0.1862)
+		(layer "F.Cu")
+		(net 399)
+	)
+	(segment
+		(start 145.5 82.4)
+		(end 146.05 82.95)
+		(width 0.1862)
+		(layer "F.Cu")
+		(net 399)
+	)
+	(segment
 		(start 145.5 80.65)
-		(end 145.5 83.1)
+		(end 145.5 82.4)
+		(width 0.1862)
+		(layer "F.Cu")
+		(net 399)
+	)
+	(segment
+		(start 146.05 82.95)
+		(end 146.45 83.35)
+		(width 0.1862)
+		(layer "F.Cu")
+		(net 399)
+	)
+	(segment
+		(start 146.45 83.8)
+		(end 146.45 84.25)
+		(width 0.1862)
+		(layer "F.Cu")
+		(net 399)
+	)
+	(segment
+		(start 148.1 85.9)
+		(end 148.2 86)
+		(width 0.1862)
+		(layer "F.Cu")
+		(net 399)
+	)
+	(segment
+		(start 146.45 83.35)
+		(end 146.45 83.8)
 		(width 0.1862)
 		(layer "F.Cu")
@@
 	)
 	(segment
-		(start 140.12 80.43)
-		(end 140.12 83.83)
-		(width 0.1862)
-		(layer "F.Cu")
-		(net 404)
-	)
-	(segment
 		(start 141.1 79.45)
 		(end 140.12 80.43)
@@
 	)
 	(segment
+		(start 140.12 80.43)
+		(end 140.12 82.22)
+		(width 0.1862)
+		(layer "F.Cu")
+		(net 404)
+	)
+	(segment
 		(start 146.7 79.45)
 		(end 146.7 79)
@@
 	)
 	(segment
+		(start 143.4 84.45)
+		(end 145.5 84.45)
+		(width 0.1862)
+		(layer "F.Cu")
+		(net 409)
+	)
+	(segment
+		(start 140.66 81.71)
+		(end 143.4 84.45)
+		(width 0.1862)
+		(layer "F.Cu")
+		(net 409)
+	)
+	(segment
+		(start 147.25 86.2)
+		(end 147.25 86.45)
+		(width 0.1862)
+		(layer "F.Cu")
+		(net 409)
+	)
+	(segment
 		(start 140.66 80.69)
-		(end 140.66 83.89)
+		(end 140.66 81.71)
+		(width 0.1862)
+		(layer "F.Cu")
+		(net 409)
+	)
+	(segment
+		(start 145.5 84.45)
+		(end 147.25 86.2)
 		(width 0.1862)
 		(layer "F.Cu")
@@
 	)
 	(segment
-		(start 149.55 76.777814)
-		(end 145.75 80.577814)
-		(width 0.1308)
-		(layer "In2.Cu")
-		(net 412)
-	)
-	(segment
 		(start 149.55 76.7)
 		(end 149.55 76.777814)
@@
 	)
 	(segment
-		(start 145.75 80.577814)
+		(start 149.55 76.7)
+		(end 149.37 76.7)
+		(width 0.1308)
+		(layer "In2.Cu")
+		(net 412)
+	)
+	(segment
+		(start 147.35 79.04)
+		(end 145.75 80.64)
+		(width 0.1308)
+		(layer "In2.Cu")
+		(net 412)
+	)
+	(segment
+		(start 147.35 78.72)
+		(end 147.35 79.04)
+		(width 0.1308)
+		(layer "In2.Cu")
+		(net 412)
+	)
+	(segment
+		(start 145.75 80.64)
 		(end 145.75 82)
+		(width 0.1308)
+		(layer "In2.Cu")
+		(net 412)
+	)
+	(segment
+		(start 149.37 76.7)
+		(end 147.35 78.72)
 		(width 0.1308)
 		(layer "In2.Cu")
@@
 	(segment
 		(start 154.4559 82.4)
-		(end 153.3559 83.5)
+		(end 154.4559 86.3)
 		(width 0.1862)
 		(layer "F.Cu")
@@
 	)
 	(segment
-		(start 153.98 82.03)
-		(end 153.01 83)
+		(start 153.25 82.76)
+		(end 153.25 86.4)
 		(width 0.1862)
 		(layer "F.Cu")
@@
 		(width 0.1862)
 		(layer "F.Cu")
+		(net 428)
+	)
+	(segment
+		(start 153.98 82.03)
+		(end 153.25 82.76)
+		(width 0.1862)
+		(layer "F.Cu")

Commit message: frouting DDR to the FPGA
Routing:
- net /Artix 7 Banks/DDR_DQ10: track 19.9 -> 32.6 mm
- net /Artix 7 Banks/DDR_DQ8: track 22.5 -> 34.3 mm
- net /Artix 7 Banks/DDR_CKE: track 16.6 -> 27.2 mm
- net /Artix 7 Banks/DDR_DQ9: track 6.55 -> 16.4 mm
- net /Artix 7 Banks/DDR_CLK+: track 14.7 -> 23.6 mm
- net /Artix 7 Banks/DDR_CLK-: track 14.7 -> 23.6 mm
- net /Artix 7 Banks/DDR_A8: track 9.00 -> 14.5 mm
- net /Artix 7 Banks/DDR_A9: track 5.46 -> 10.5 mm
- net /Artix 7 Banks/DDR_A7: track 3.77 -> 8.36 mm
- net /Artix 7 Banks/~{DDR_ODT}: track 9.63 -> 13.8 mm
- net unconnected-(U1C-IO_L18N_T2_34-PadAA6): track 0.00 -> 1.71 mm, vias 0 -> 1
- net unconnected-(U1C-IO_L9N_T1_DQS_34-PadAA3): track 0.00 -> 1.66 mm, vias 0 -> 1
- net unconnected-(U1C-IO_L11N_T1_SRCC_34-PadAA4): track 0.00 -> 0.79 mm, vias 0 -> 1
- net unconnected-(U1C-IO_L9P_T1_DQS_34-PadY3): track 0.00 -> 0.71 mm, vias 0 -> 1
- net unconnected-(U1C-IO_L7P_T1_34-PadAA1): track 0.00 -> 0.71 mm, vias 0 -> 1
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
Commit message: more IO routing
Parts:
- moved C155 0.10 mm to (153.3, 91.2)
Routing:
- net /Artix 7 Banks/DDR_DQ1: track 11.4 -> 25.1 mm
- net /Artix 7 Banks/DDR_DQM0: track 10.9 -> 23.6 mm
- net /Artix 7 Banks/DDR_DQM1: track 5.46 -> 17.2 mm
- net /Artix 7 Banks/DDR_DQS0+: track 9.69 -> 19.8 mm
- net /Artix 7 Banks/DDR_A6: track 8.85 -> 18.9 mm
- net /Artix 7 Banks/~{DDR_CAS}: track 3.54 -> 13.3 mm
- net /Artix 7 Banks/DDR_DQS0-: track 10.6 -> 20.2 mm
- net /Artix 7 Banks/DDR_DQ0: track 3.73 -> 13.3 mm
- net /Artix 7 Banks/DDR_A12: track 6.93 -> 16.0 mm
- net /Artix 7 Banks/DDR_DQ5: track 13.7 -> 22.7 mm
- net /Artix 7 Banks/DDR_DQ10: track 32.6 -> 41.4 mm
- net /Artix 7 Banks/~{DDR_RAS}: track 4.01 -> 12.7 mm
- net /Artix 7 Banks/DDR_DQ11: track 3.76 -> 12.3 mm
- net /Artix 7 Banks/DDR_A5: track 3.58 -> 11.6 mm
- net /Artix 7 Banks/DDR_DQ9: track 16.4 -> 8.78 mm
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
Commit message: routed top and inner DDR, working on bottom!
Routing:
- net /Artix 7 Banks/DDR_DQ9: track 8.78 -> 23.1 mm
- net /Artix 7 Banks/DDR_A7: track 2.93 -> 15.2 mm
- net /Artix 7 Banks/DDR_A8: track 7.51 -> 18.5 mm
- net /Artix 7 Banks/~{DDR_ODT}: track 10.9 -> 19.8 mm
- net /Artix 7 Banks/DDR_A9: track 4.25 -> 10.6 mm
- net /Artix 7 Banks/DDR_DQ8: track 41.6 -> 46.3 mm
- net /Artix 7 Banks/DDR_A4: track 13.9 -> 17.9 mm
- net /Artix 7 Banks/DDR_A6: track 18.9 -> 18.2 mm
