File: PCB/banks.kicad_sch (KiCad schematic)
At the start: 8 parts, among them U1 XC7A50T-FGG484, Y3 100MHz

Commit message: cleaned up the schematic to look cooler
Changed lines of the file:
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@@
-		)
-	)
-	(hierarchical_label "{EPHY}"
-		(shape bidirectional)
-		(at 400.05 71.12 0)
-		(effects
-			(font
-				(size 1.27 1.27)
-			)
-			(justify left)
 		)
 	)

Commit message: forgot to add decouping to my banks
Parts:
- added C124, C125, C135, C136, C137, C138, C143, C144, C145, C146, C91, C92: 470n, Capacitor_SMD:C_0201_0603Metric, symbol Device:C
- added C132, C140, C88: 47u, Capacitor_SMD:C_1206_3216Metric, symbol Device:C
- added C133, C134, C141, C142, C89, C90: 4u7, Capacitor_SMD:C_0603_1608Metric, symbol Device:C
Connections:
- net +3V3: now also C124.1, C125.1, C132.1, C133.1, C134.1, C135.1, C136.1, C137.1, C138.1, C140.1, C141.1, C142.1, C143.1, C144.1, C145.1, C146.1, C88.1, C89.1, C90.1, C91.1, C92.1
- net GND: now also C124.2, C125.2, C132.2, C133.2, C134.2, C135.2, C136.2, C137.2, C138.2, C140.2, C141.2, C142.2, C143.2, C144.2, C145.2, C146.2, C88.2, C89.2, C90.2, C91.2, C92.2
Other:
- note added: "47u + 2x 4u7 + 4x 470n capacitors per bank!"

Commit message: wired decoupling to banks 34 and 35
Parts:
- added C149, C158: 47u, Capacitor_SMD:C_1206_3216Metric, symbol Device:C
- added C152, C153, C159, C160: 4u7, Capacitor_SMD:C_0603_1608Metric, symbol Device:C
- added C154, C155, C156, C157, C161, C162, C163, C164: 470n, Capacitor_SMD:C_0201_0603Metric, symbol Device:C
Connections:
- net GND: now also C149.2, C152.2, C153.2, C154.2, C155.2, C156.2, C157.2, C158.2, C159.2, C160.2, C161.2, C162.2, C163.2, C164.2
- net +1V5: now reaches U1.AA7 (VCCO_34)
- net +1V5: now also U1.AB4 (VCCO_34), U1.C1 (VCCO_35), U1.F2 (VCCO_35), U1.H6 (VCCO_35), U1.J3 (VCCO_35), U1.M4 (VCCO_35), U1.N1 (VCCO_35), U1.R5 (VCCO_34), U1.T2 (VCCO_34), U1.V6 (VCCO_34), U1.W3 (VCCO_34), C149.1, C152.1, C153.1, C154.1, C155.1, C156.1, C157.1, C158.1, C159.1, C160.1, C161.1, C162.1, C163.1, C164.1
Other:
- moved on the sheet: C140, C141, C142, C143, C144, C145, C146, U1B, U1C

Commit message: wired up bank 16
Parts:
- added C165: 47u, Capacitor_SMD:C_1206_3216Metric, symbol Device:C
- added C166, C167: 4u7, Capacitor_SMD:C_0603_1608Metric, symbol Device:C
- added C168, C169, C170, C171: 470n, Capacitor_SMD:C_0201_0603Metric, symbol Device:C
Connections:
- net +3V3: now also U1.A17 (VCCO_16), U1.B14 (VCCO_16), U1.C21 (VCCO_16), U1.D18 (VCCO_16), U1.E15 (VCCO_16), U1.F22 (VCCO_16), C165.1, C166.1, C167.1, C168.1, C169.1, C170.1, C171.1
- net GND: now also C165.2, C166.2, C167.2, C168.2, C169.2, C170.2, C171.2

Commit message: doing a lot more routing
Connections:
- net DDR_DQS1-: now reaches U1.AA3 (IO_L9N_T1_DQS_34)
- net DDR_DQS0-: now reaches U1.V8 (IO_L21N_T3_DQS_34)
- net DDR_DQS0+: now reaches U1.V9 (IO_L21P_T3_DQS_34)
- net DDR_DQS1+: now reaches U1.Y3 (IO_L9P_T1_DQS_34)
- net DDR_CLK-: now reaches U1.Y7 (IO_L23N_T3_34)
- net DDR_CLK+: now reaches U1.Y8 (IO_L23P_T3_34)

Commit message: starting to actually put the DDR traces to their pins
Connections:
- net DDR_DQ2: now reaches U1.AA5 (IO_L10P_T1_34)
- net DDR_DQ15: now reaches U1.AA6 (IO_L18N_T2_34)
- net DDR_DQ13: now reaches U1.AB5 (IO_L10N_T1_34)
- net DDR_DQ14: now reaches U1.AB6 (IO_L20N_T3_34)
- net DDR_DQ12: now reaches U1.AB7 (IO_L20P_T3_34)
- net DDR_DQ1: now reaches U1.P6 (IO_L24P_T3_35)
- net DDR_DQ10: now reaches U1.R6 (IO_L17P_T2_34)
- net DDR_DQ7: now reaches U1.T5 (IO_L14P_T2_SRCC_34)
- net DDR_DQM0: now reaches U1.T6 (IO_L17N_T2_34)
- net DDR_DQ11: now reaches U1.U6 (IO_L16P_T2_34)
- net DDR_DQ6: now reaches U1.V4 (IO_L12P_T1_MRCC_34)
- net DDR_DQ9: now reaches U1.V5 (IO_L16N_T2_34)
- net DDR_DQ5: now reaches U1.V7 (IO_L19P_T3_34)
- net DDR_DQ8: now reaches U1.W6 (IO_L15P_T2_DQS_34)
- net DDR_DQ4: now reaches U1.W7 (IO_L19N_T3_VREF_34)
- net DDR_DQ0: now reaches U1.Y9 (IO_L24N_T3_34)

Commit message: a bunch more routing and assigning, really messy but coming along
Connections:
- net DDR_BA0: now reaches U1.AA4 (IO_L11N_T1_SRCC_34)
- net DDR_A12: now reaches U1.AA8 (IO_L22P_T3_34)
- net DDR_A14: now reaches U1.AB1 (IO_L7N_T1_34)
- net ~{DDR_RESET}: now reaches U1.AB2 (IO_L8N_T1_34)
- net ~{DDR_WE}: now reaches U1.AB3 (IO_L8P_T1_34)
- net DDR_A10: now reaches U1.AB8 (IO_L22N_T3_34)
- net DDR_A9: now reaches U1.R2 (IO_L3N_T0_DQS_34)
- net DDR_A6: now reaches U1.T1 (IO_L1P_T0_34)
- net DDR_BA2: now reaches U1.T3 (IO_0_34)
- net DDR_A1: now reaches U1.U1 (IO_L1N_T0_34)
- net DDR_A4: now reaches U1.U2 (IO_L2P_T0_34)
- net DDR_A5: now reaches U1.U3 (IO_L6P_T0_34)
- net ~{DDR_ODT}: now reaches U1.V3 (IO_L6N_T0_VREF_34)
- net DDR_A11: now reaches U1.W1 (IO_L5P_T0_34)
- net DDR_A7: now reaches U1.W2 (IO_L4P_T0_34)
- net DDR_A3: now reaches U1.W4 (IO_L12N_T1_MRCC_34)
- net DDR_CKE: now reaches U1.W5 (IO_L15N_T2_DQS_34)
- net DDR_DQM1: now reaches U1.W9 (IO_L24P_T3_34)
- net DDR_A13: now reaches U1.Y1 (IO_L5N_T0_34)
- net DDR_A2: now reaches U1.Y2 (IO_L4N_T0_34)
- net DDR_A0: now reaches U1.Y4 (IO_L11P_T1_SRCC_34)
- net ~{DDR_CAS}: now reaches U1.Y6 (IO_L18P_T2_34)
- no-connect marks 10 -> 17
Other:
- moved on the sheet: C149, C152, C153, C154, C155, C156, C157, C158, C159, C160, C161, C162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

Commit message: finished routing all the pins, very messy still
Connections:
- net DDR_A9: now also U1.R3 (IO_L3P_T0_DQS_34); no longer U1.R2 (IO_L3N_T0_DQS_34)
- net ~{DDR_RAS}: now reaches U1.T4 (IO_L13N_T2_MRCC_34)
- new net DDR_A8: U1.R2 (IO_L3N_T0_DQS_34)
- no-connect marks 17 -> 14
Changed lines of the file:
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@@
 	)
 	(no_connect
-		(at 702.31 102.87)
-	)
-	(no_connect
 		(at 261.62 209.55)
 	)
@@
 	)
 	(no_connect
-		(at 702.31 156.21)
-	)
-	(no_connect
 		(at 702.31 214.63)
 	)
@@
 	)
 	(no_connect
-		(at 702.31 100.33)
-	)
-	(no_connect
 		(at 127 113.03)
 	)
@@
 	)
 	(bus_entry
+		(at 647.7 153.67)
+		(size 2.54 2.54)
+		(stroke
+			(width 0)
+			(type default)
+		)
+	)
+	(bus_entry
 		(at 622.3 168.91)
 		(size 2.54 2.54)
@@
 	)
 	(bus_entry
+		(at 674.37 100.33)
+		(size 2.54 2.54)
+		(stroke
+			(width 0)
+			(type default)
+		)
+	)
+	(bus_entry
 		(at 622.3 179.07)
 		(size 2.54 2.54)
@@
 	)
 	(bus_entry
+		(at 674.37 102.87)
+		(size 2.54 2.54)
+		(stroke
+			(width 0)
+			(type default)
+		)
+	)
+	(bus_entry
 		(at 674.37 87.63)
 		(size 2.54 2.54)
@@
 	(bus
 		(pts
-			(xy 674.37 95.25) (xy 674.37 102.87)
+			(xy 674.37 95.25) (xy 674.37 100.33)
 		)
 		(stroke
@@
 		)
 	)
+	(bus
+		(pts
+			(xy 647.7 153.67) (xy 647.7 165.1)
+		)
+		(stroke
+			(width 0)
+			(type default)
+		)
+	)
 	(wire
 		(pts
@@
 	(wire
 		(pts
+			(xy 650.24 156.21) (xy 702.31 156.21)
+		)
+		(stroke
+			(width 0)
+			(type default)
+		)
+	)
+	(wire
+		(pts
 			(xy 125.73 49.53) (xy 125.73 52.07)
 		)
@@
 	(bus
 		(pts
-			(xy 647.7 128.27) (xy 647.7 165.1)
+			(xy 647.7 128.27) (xy 647.7 153.67)
 		)
 		(stroke
@@
 	(wire
 		(pts
+			(xy 676.91 102.87) (xy 702.31 102.87)
+		)
+		(stroke
+			(width 0)
+			(type default)
+		)
+	)
+	(wire
+		(pts
 			(xy 281.94 68.58) (xy 281.94 69.85)
 		)
@@
 		)
 	)
+	(bus
+		(pts
+			(xy 674.37 100.33) (xy 674.37 102.87)
+		)
+		(stroke
+			(width 0)
+			(type default)
+		)
+	)
 	(wire
 		(pts
@@
 		)
 	)
+	(label "~{DDR_RAS}"
+		(at 662.94 156.21 180)
+		(effects
+			(font
+				(size 1.27 1.27)
+			)
+			(justify right bottom)
+		)
+	)
 	(label "DDR_DQS1+"
 		(at 638.81 133.35 180)
@@
 		)
 	)
-	(label "DDR_A9"
-		(at 687.07 105.41 180)
-		(effects
-			(font
-				(size 1.27 1.27)
-			)
-			(justify right bottom)
-		)
-	)
 	(label "~{PCIe_PEWAKE}"
 		(at 175.26 168.91 180)
@@
 		)
 	)
+	(label "DDR_A8"
+		(at 687.07 105.41 180)
+		(effects
+			(font
+				(size 1.27 1.27)
+			)
+			(justify right bottom)
+		)
+	)
 	(label "DDR_DQ4"
 		(at 638.81 186.69 180)
@@
 		)
 	)
+	(label "DDR_A9"
+		(at 687.07 102.87 180)
+		(effects
+			(font
+				(size 1.27 1.27)
+			)
+			(justify right bottom)
+		)
+	)
 	(hierarchical_label "{PCIe_COMMAND}"
 		(shape bidirectional)
@@
 		(lib_id "Device:C")
 		(at 741.68 55.88 0)
+		(mirror y)
 		(unit 1)
 		(exclude_from_sim no)
@@
 		(dnp no)
 		(property "Reference" "C154"
-			(at 742.696 52.832 0)
+			(at 740.664 52.832 0)
 			(effects
 				(font
@@
 		)
 		(property "Value" "470n"
-			(at 742.696 58.928 0)
+			(at 740.664 58.928 0)
 			(effects
 				(font
@@
 		)
 		(property "Footprint" "Capacitor_SMD:C_0201_0603Metric"
-			(at 742.6452 59.69 0)
+			(at 740.7148 59.69 0)
 			(effects
 				(font
