File: PCB/banks.kicad_sch (KiCad schematic)
At the start: 50 parts, among them U1 XC7A50T-FGG484, Y3 100MHz

Commit message: almost done vivado memory verification
Connections:
- net DDR_DQ1: now also U1.R4 (IO_L13P_T2_MRCC_34); no longer U1.P6 (IO_L24P_T3_35)
Other:
- note added: "Sus A14 >"
Changed lines of the file:
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@@
 		)
 	)
+	(text "Sus A14 >"
+		(exclude_from_sim no)
+		(at 607.568 122.682 0)
+		(effects
+			(font
+				(size 2.54 2.54)
+			)
+		)
+	)
 	(text "Wait for rails before starting the crystal! >"
 		(exclude_from_sim no)
@@
 	)
 	(no_connect
-		(at 702.31 153.67)
-	)
-	(no_connect
 		(at 260.35 166.37)
 	)
@@
 	)
 	(no_connect
+		(at 702.31 100.33)
+	)
+	(no_connect
 		(at 127 105.41)
 	)
@@
 	)
 	(bus_entry
-		(at 647.7 153.67)
+		(at 647.7 154.94)
 		(size 2.54 2.54)
 		(stroke
@@
 	)
 	(bus_entry
+		(at 622.3 151.13)
+		(size 2.54 2.54)
+		(stroke
+			(width 0)
+			(type default)
+		)
+	)
+	(bus_entry
 		(at 622.3 171.45)
 		(size 2.54 2.54)
@@
 	)
 	(bus_entry
-		(at 817.88 207.01)
-		(size -2.54 2.54)
-		(stroke
-			(width 0)
-			(type default)
-		)
-	)
-	(bus_entry
 		(at 622.3 189.23)
 		(size 2.54 2.54)
@@
 	(wire
 		(pts
-			(xy 803.91 209.55) (xy 815.34 209.55)
-		)
-		(stroke
-			(width 0)
-			(type default)
-		)
-	)
-	(wire
-		(pts
 			(xy 156.21 62.23) (xy 156.21 59.69)
 		)
@@
 	(bus
 		(pts
-			(xy 824.23 207.01) (xy 817.88 207.01)
-		)
-		(stroke
-			(width 0)
-			(type default)
-		)
-	)
-	(bus
-		(pts
 			(xy 647.7 118.11) (xy 647.7 125.73)
 		)
@@
 	(bus
 		(pts
-			(xy 622.3 146.05) (xy 622.3 156.21)
+			(xy 622.3 146.05) (xy 622.3 151.13)
 		)
 		(stroke
@@
 	(bus
 		(pts
-			(xy 647.7 153.67) (xy 647.7 165.1)
+			(xy 647.7 154.94) (xy 647.7 165.1)
 		)
 		(stroke
@@
 	(wire
 		(pts
-			(xy 650.24 156.21) (xy 702.31 156.21)
+			(xy 650.24 157.48) (xy 651.51 157.48)
 		)
 		(stroke
@@
 	(bus
 		(pts
-			(xy 647.7 128.27) (xy 647.7 153.67)
+			(xy 647.7 128.27) (xy 647.7 154.94)
 		)
 		(stroke
@@
 	(wire
 		(pts
+			(xy 651.51 156.21) (xy 702.31 156.21)
+		)
+		(stroke
+			(width 0)
+			(type default)
+		)
+	)
+	(wire
+		(pts
 			(xy 350.52 68.58) (xy 350.52 69.85)
 		)
@@
 	(wire
 		(pts
+			(xy 651.51 157.48) (xy 651.51 156.21)
+		)
+		(stroke
+			(width 0)
+			(type default)
+		)
+	)
+	(wire
+		(pts
 			(xy 156.21 49.53) (xy 156.21 52.07)
 		)
@@
 	(wire
 		(pts
+			(xy 624.84 153.67) (xy 702.31 153.67)
+		)
+		(stroke
+			(width 0)
+			(type default)
+		)
+	)
+	(wire
+		(pts
 			(xy 345.44 68.58) (xy 345.44 69.85)
 		)
@@
 	(bus
 		(pts
+			(xy 622.3 151.13) (xy 622.3 156.21)
+		)
+		(stroke
+			(width 0)
+			(type default)
+		)
+	)
+	(bus
+		(pts
 			(xy 179.07 166.37) (xy 179.07 168.91)
 		)
@@
 		)
 	)
-	(bus
-		(pts
-			(xy 817.88 207.01) (xy 817.88 218.44)
-		)
-		(stroke
-			(width 0)
-			(type default)
-		)
-	)
 	(wire
 		(pts
@@
 		)
 	)
+	(label "DDR_DQ1"
+		(at 638.81 153.67 180)
+		(effects
+			(font
+				(size 1.27 1.27)
+			)
+			(justify right bottom)
+		)
+	)
 	(label "QSPI_DQ3"
 		(at 140.97 100.33 180)
@@
 		)
 	)
-	(label "DDR_DQ1"
-		(at 805.18 209.55 0)
-		(effects
-			(font
-				(size 1.27 1.27)
-			)
-			(justify left bottom)
-		)
-	)
 	(label "~{PCIe_CLKREQ}"
 		(at 175.26 163.83 180)
@@
 		(effects
 			(font
-				(size 1.27 1.27)
-			)
-			(justify left)
-		)
-	)
-	(hierarchical_label "{DDR_DATA}"
-		(shape bidirectional)
-		(at 824.23 207.01 0)
-		(effects
-			(font

Commit message: finally routed a little mischevious DQ3
Connections:
- net DDR_DQ1: now also U1.U7 (IO_25_34); no longer U1.R4 (IO_L13P_T2_MRCC_34)
- new net DDR_DQ3: U1.R4 (IO_L13P_T2_MRCC_34)
- no-connect marks 14 -> 13
Changed lines of the file:
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@@
 	)
 	(no_connect
-		(at 702.31 214.63)
-	)
-	(no_connect
 		(at 702.31 100.33)
 	)
@@
 	)
 	(bus_entry
+		(at 622.3 151.13)
+		(size 2.54 2.54)
+		(stroke
+			(width 0)
+			(type default)
+		)
+	)
+	(bus_entry
 		(at 622.3 209.55)
 		(size 2.54 2.54)
@@
 	)
 	(bus_entry
+		(at 622.3 212.09)
+		(size 2.54 2.54)
+		(stroke
+			(width 0)
+			(type default)
+		)
+	)
+	(bus_entry
 		(at 622.3 194.31)
 		(size 2.54 2.54)
@@
 		)
 	)
+	(bus
+		(pts
+			(xy 622.3 212.09) (xy 622.3 217.17)
+		)
+		(stroke
+			(width 0)
+			(type default)
+		)
+	)
 	(wire
 		(pts
@@
 	(wire
 		(pts
+			(xy 624.84 153.67) (xy 702.31 153.67)
+		)
+		(stroke
+			(width 0)
+			(type default)
+		)
+	)
+	(wire
+		(pts
 			(xy 712.47 46.99) (xy 712.47 49.53)
 		)
@@
 	(bus
 		(pts
-			(xy 622.3 209.55) (xy 622.3 217.17)
+			(xy 622.3 209.55) (xy 622.3 212.09)
 		)
 		(stroke
@@
 	(wire
 		(pts
+			(xy 624.84 214.63) (xy 702.31 214.63)
+		)
+		(stroke
+			(width 0)
+			(type default)
+		)
+	)
+	(wire
+		(pts
 			(xy 802.64 49.53) (xy 810.26 49.53)
 		)
@@
 	(wire
 		(pts
-			(xy 624.84 153.67) (xy 702.31 153.67)
-		)
-		(stroke
-			(width 0)
-			(type default)
-		)
-	)
-	(wire
-		(pts
 			(xy 345.44 68.58) (xy 345.44 69.85)
 		)
@@
 		)
 	)
-	(label "DDR_DQ1"
-		(at 638.81 153.67 180)
-		(effects
-			(font
-				(size 1.27 1.27)
-			)
-			(justify right bottom)
-		)
-	)
 	(label "QSPI_DQ3"
 		(at 140.97 100.33 180)
@@
 		)
 	)
+	(label "DDR_DQ1"
+		(at 638.81 214.63 180)
+		(effects
+			(font
+				(size 1.27 1.27)
+			)
+			(justify right bottom)
+		)
+	)
 	(label "DDR_A4"
 		(at 687.07 97.79 180)
@@
 		(effects
 			(font
+				(size 1.27 1.27)
+			)
+			(justify right bottom)
+		)
+	)
+	(label "DDR_DQ3"
+		(at 638.81 153.67 180)
+		(effects
+			(font

Commit message: TRYING TO GET THIS TRACE THROUGH FEHJFSHEJKF
Connections:
- net DDR_DQ1: now also U1.U5 (IO_L14N_T2_SRCC_34); no longer U1.U7 (IO_25_34)
- new net DDR_BA1: U1.U7 (IO_25_34)
- no-connect marks 13 -> 12
Changed lines of the file:
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@@
 	)
 	(no_connect
-		(at 702.31 161.29)
-	)
-	(no_connect
 		(at 127 113.03)
 	)
@@
 	)
 	(bus_entry
+		(at 674.37 213.36)
+		(size 2.54 2.54)
+		(stroke
+			(width 0)
+			(type default)
+		)
+	)
+	(bus_entry
 		(at 622.3 151.13)
 		(size 2.54 2.54)
@@
 	)
 	(bus_entry
-		(at 622.3 212.09)
-		(size 2.54 2.54)
-		(stroke
-			(width 0)
-			(type default)
-		)
-	)
-	(bus_entry
 		(at 622.3 194.31)
 		(size 2.54 2.54)
@@
 	)
 	(bus_entry
+		(at 622.3 158.75)
+		(size 2.54 2.54)
+		(stroke
+			(width 0)
+			(type default)
+		)
+	)
+	(bus_entry
 		(at 622.3 146.05)
 		(size 2.54 2.54)
@@
 		)
 	)
-	(bus
-		(pts
-			(xy 674.37 200.66) (xy 674.37 217.17)
-		)
-		(stroke
-			(width 0)
-			(type default)
-		)
-	)
 	(wire
 		(pts
@@
 		)
 	)
-	(bus
-		(pts
-			(xy 622.3 212.09) (xy 622.3 217.17)
-		)
-		(stroke
-			(width 0)
-			(type default)
-		)
-	)
 	(wire
 		(pts
@@
 	(bus
 		(pts
+			(xy 622.3 158.75) (xy 622.3 161.29)
+		)
+		(stroke
+			(width 0)
+			(type default)
+		)
+	)
+	(bus
+		(pts
 			(xy 674.37 102.87) (xy 674.37 105.41)
 		)
@@
 		)
 	)
+	(bus
+		(pts
+			(xy 674.37 213.36) (xy 674.37 214.63)
+		)
+		(stroke
+			(width 0)
+			(type default)
+		)
+	)
 	(wire
 		(pts
@@
 	(wire
 		(pts
+			(xy 678.18 215.9) (xy 678.18 214.63)
+		)
+		(stroke
+			(width 0)
+			(type default)
+		)
+	)
+	(wire
+		(pts
 			(xy 717.55 68.58) (xy 717.55 69.85)
 		)
@@
 	(bus
 		(pts
-			(xy 622.3 156.21) (xy 622.3 161.29)
+			(xy 622.3 156.21) (xy 622.3 158.75)
 		)
 		(stroke
@@
 		)
 	)
-	(bus
-		(pts
-			(xy 622.3 209.55) (xy 622.3 212.09)
-		)
-		(stroke
-			(width 0)
-			(type default)
-		)
-	)
 	(wire
 		(pts
@@
 		)
 	)
+	(bus
+		(pts
+			(xy 674.37 200.66) (xy 674.37 213.36)
+		)
+		(stroke
+			(width 0)
+			(type default)
+		)
+	)
 	(wire
 		(pts
@@
 	(wire
 		(pts
+			(xy 676.91 215.9) (xy 678.18 215.9)
+		)
+		(stroke
+			(width 0)
+			(type default)
+		)
+	)
+	(wire
+		(pts
 			(xy 384.81 49.53) (xy 392.43 49.53)
 		)
@@
 	(wire
 		(pts
-			(xy 624.84 214.63) (xy 702.31 214.63)
-		)
-		(stroke
-			(width 0)
-			(type default)
-		)
-	)
-	(wire
-		(pts
 			(xy 802.64 49.53) (xy 810.26 49.53)
 		)
@@
 		)
 	)
+	(wire
+		(pts
+			(xy 624.84 161.29) (xy 702.31 161.29)
+		)
+		(stroke
+			(width 0)
+			(type default)
+		)
+	)
 	(bus
 		(pts
@@
 		)
 	)
+	(wire
+		(pts
+			(xy 678.18 214.63) (xy 702.31 214.63)
+		)
+		(stroke
+			(width 0)
+			(type default)
+		)
+	)
 	(bus
 		(pts
@@
 		)
 	)
-	(label "DDR_DQ1"
-		(at 638.81 214.63 180)
+	(label "DDR_BA1"
+		(at 688.34 214.63 180)
 		(effects
 			(font
@@
 		(effects
 			(font
+				(size 1.27 1.27)
+			)
+			(justify right bottom)
+		)
+	)
+	(label "DDR_DQ1"
+		(at 638.81 161.29 180)
+		(effects
+			(font

Commit message: a bunch of wiring
Connections:
- net DDR_DQ13 is gone; now on net DDR_BA0: U1.AB5 (IO_L10N_T1_34)
- net DDR_DQ6 is gone; now on net DDR_DQ9: U1.V4 (IO_L12P_T1_MRCC_34)
- net DDR_A0: now also U1.U3 (IO_L6P_T0_34); no longer U1.Y4 (IO_L11P_T1_SRCC_34)
- net DDR_A1: now also U1.AB2 (IO_L8N_T1_34); no longer U1.U1 (IO_L1N_T0_34)
- net DDR_A11: now also U1.Y1 (IO_L5N_T0_34); no longer U1.W1 (IO_L5P_T0_34)
- net DDR_A13: now also U1.AA1 (IO_L7P_T1_34); no longer U1.Y1 (IO_L5N_T0_34)
- net DDR_A2: now also U1.U1 (IO_L1N_T0_34); no longer U1.Y2 (IO_L4N_T0_34)
- net DDR_A5: now also U1.Y2 (IO_L4N_T0_34); no longer U1.U3 (IO_L6P_T0_34)
- net DDR_A9: now also U1.W1 (IO_L5P_T0_34); no longer U1.R3 (IO_L3P_T0_DQS_34)
- net DDR_BA0: no longer U1.AA4 (IO_L11N_T1_SRCC_34)
- net DDR_BA1: now also U1.T3 (IO_0_34); no longer U1.U7 (IO_25_34)
- net DDR_BA2: now also U1.Y4 (IO_L11P_T1_SRCC_34); no longer U1.T3 (IO_0_34)
- net DDR_DQ9: no longer U1.V5 (IO_L16N_T2_34)
- net ~{DDR_RESET}: now also U1.AB3 (IO_L8P_T1_34); no longer U1.AB2 (IO_L8N_T1_34)
- net ~{DDR_WE}: now also U1.AA4 (IO_L11N_T1_SRCC_34); no longer U1.AB3 (IO_L8P_T1_34)
- net DDR_A10: no longer names the net of U1.AB8 (IO_L22N_T3_34)
- net DDR_A12: no longer names the net of U1.AA8 (IO_L22P_T3_34)
- net DDR_A3: no longer names the net of U1.W4 (IO_L12N_T1_MRCC_34)
- net DDR_CKE: no longer names the net of U1.W5 (IO_L15N_T2_DQS_34)
- net DDR_CLK+: no longer names the net of U1.Y8 (IO_L23P_T3_34)
- net DDR_CLK-: no longer names the net of U1.Y7 (IO_L23N_T3_34)
- net DDR_DQ0: no longer names the net of U1.Y9 (IO_L24N_T3_34)
- net DDR_DQ1: no longer names the net of U1.U5 (IO_L14N_T2_SRCC_34)
- net DDR_DQ10: no longer names the net of U1.R6 (IO_L17P_T2_34)
- net DDR_DQ11: no longer names the net of U1.U6 (IO_L16P_T2_34)
- net DDR_DQ12: no longer names the net of U1.AB7 (IO_L20P_T3_34)
- net DDR_DQ14: no longer names the net of U1.AB6 (IO_L20N_T3_34)
- net DDR_DQ15: no longer names the net of U1.AA6 (IO_L18N_T2_34)
- net DDR_DQ3: no longer names the net of U1.R4 (IO_L13P_T2_MRCC_34)
- net DDR_DQ4: no longer names the net of U1.W7 (IO_L19N_T3_VREF_34)
- net DDR_DQ5: no longer names the net of U1.V7 (IO_L19P_T3_34)
- net DDR_DQ7: no longer names the net of U1.T5 (IO_L14P_T2_SRCC_34)
- net DDR_DQ8: no longer names the net of U1.W6 (IO_L15P_T2_DQS_34)
- net DDR_DQM0: no longer names the net of U1.T6 (IO_L17N_T2_34)
- net DDR_DQM1: no longer names the net of U1.W9 (IO_L24P_T3_34)
- net DDR_DQS0+: no longer names the net of U1.V9 (IO_L21P_T3_DQS_34)
- net DDR_DQS0-: no longer names the net of U1.V8 (IO_L21N_T3_DQS_34)
- net ~{DDR_CAS}: no longer names the net of U1.Y6 (IO_L18P_T2_34)
- net ~{DDR_RAS}: no longer names the net of U1.T4 (IO_L13N_T2_MRCC_34)

Commit message: finished wiring
Connections:
- net DDR_DQS1-: now also U1.V8 (IO_L21N_T3_DQS_34)
- net DDR_DQ15: now reaches U1.AA6 (IO_L18N_T2_34)
- net DDR_DQ12: now reaches U1.AA8 (IO_L22P_T3_34)
- net DDR_DQ13: now reaches U1.AB6 (IO_L20N_T3_34)
- net DDR_DQ14: now reaches U1.AB7 (IO_L20P_T3_34)
- net DDR_A10: now reaches U1.AB8 (IO_L22N_T3_34)
- net DDR_DQ10: now reaches U1.R6 (IO_L17P_T2_34)
- net ~{DDR_RAS}: now reaches U1.T4 (IO_L13N_T2_MRCC_34)
- net DDR_DQ7: now reaches U1.T5 (IO_L14P_T2_SRCC_34)
- net DDR_DQ1: now reaches U1.T6 (IO_L17N_T2_34)
- net DDR_DQ1: now also U1.U5 (IO_L14N_T2_SRCC_34)
- net DDR_DQ4: now reaches U1.U6 (IO_L16P_T2_34)
- net ~{DDR_CAS}: now reaches U1.V5 (IO_L16N_T2_34)
- net DDR_DQ5: now reaches U1.V7 (IO_L19P_T3_34)
- net DDR_DQS0+: now reaches U1.V9 (IO_L21P_T3_DQS_34)
- net DDR_A3: now reaches U1.W4 (IO_L12N_T1_MRCC_34)
- net DDR_CKE: now reaches U1.W5 (IO_L15N_T2_DQS_34)
- net DDR_DQ8: now reaches U1.W6 (IO_L15P_T2_DQS_34)
- net DDR_DQ6: now reaches U1.W7 (IO_L19N_T3_VREF_34)
- net DDR_DQM1: now reaches U1.W9 (IO_L24P_T3_34)
- net DDR_A12: now reaches U1.Y6 (IO_L18P_T2_34)
- net DDR_CLK-: now reaches U1.Y7 (IO_L23N_T3_34)
- net DDR_CLK+: now reaches U1.Y8 (IO_L23P_T3_34)
- net DDR_DQ0: now reaches U1.Y9 (IO_L24N_T3_34)
- no-connect marks 12 -> 14

Commit message: a bunch of routing
Connections:
- net DDR_DQ1: no longer U1.U5 (IO_L14N_T2_SRCC_34)
- net DDR_DQS1-: no longer U1.V8 (IO_L21N_T3_DQS_34)
- net DDR_DQ3: now reaches U1.R3 (IO_L3P_T0_DQS_34)
- net DDR_DQM0: now reaches U1.R4 (IO_L13P_T2_MRCC_34)
- new net DDR_DQ11: U1.U5 (IO_L14N_T2_SRCC_34)
- new net DDR_DQS0-: U1.V8 (IO_L21N_T3_DQS_34)
- no-connect marks 14 -> 12
Changed lines of the file:
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@@
 	)
 	(no_connect
-		(at 702.31 153.67)
-	)
-	(no_connect
 		(at 702.31 214.63)
 	)
@@
 	)
 	(no_connect
-		(at 702.31 102.87)
-	)
-	(no_connect
 		(at 127 105.41)
 	)
@@
 	)
 	(bus_entry
+		(at 622.3 151.13)
+		(size 2.54 2.54)
+		(stroke
+			(width 0)
+			(type default)
+		)
+	)
+	(bus_entry
 		(at 674.37 140.97)
 		(size 2.54 2.54)
@@
 	)
 	(bus_entry
+		(at 622.3 99.06)
+		(size 2.54 2.54)
+		(stroke
+			(width 0)
+			(type default)
+		)
+	)
+	(bus_entry
 		(at 622.3 132.08)
 		(size 2.54 2.54)
@@
 	)
 	(bus_entry
+		(at 622.3 158.75)
+		(size 2.54 2.54)
+		(stroke
+			(width 0)
+			(type default)
+		)
+	)
+	(bus_entry
+		(at 622.3 158.75)
+		(size 2.54 2.54)
+		(stroke
+			(width 0)
+			(type default)
+		)
+	)
+	(bus_entry
 		(at 647.7 142.24)
 		(size 2.54 2.54)
@@
 	)
 	(bus_entry
+		(at 622.3 194.31)
+		(size 2.54 2.54)
+		(stroke
+			(width 0)
+			(type default)
+		)
+	)
+	(bus_entry
 		(at 647.7 153.67)
 		(size 2.54 2.54)
@@
 	(wire
 		(pts
+			(xy 676.91 101.6) (xy 676.91 102.87)
+		)
+		(stroke
+			(width 0)
+			(type default)
+		)
+	)
+	(wire
+		(pts
 			(xy 346.71 62.23) (xy 354.33 62.23)
 		)
@@
 	(bus
 		(pts
-			(xy 622.3 144.78) (xy 622.3 156.21)
+			(xy 622.3 144.78) (xy 622.3 151.13)
 		)
 		(stroke
@@
 	(wire
 		(pts
+			(xy 647.7 153.67) (xy 702.31 153.67)
+		)
+		(stroke
+			(width 0)
+			(type default)
+		)
+	)
+	(wire
+		(pts
 			(xy 133.35 62.23) (xy 133.35 59.69)
 		)
@@
 	(bus
 		(pts
+			(xy 622.3 99.06) (xy 622.3 129.54)
+		)
+		(stroke
+			(width 0)
+			(type default)
+		)
+	)
+	(bus
+		(pts
 			(xy 144.78 80.01) (xy 153.67 80.01)
 		)
@@
 	(wire
 		(pts
-			(xy 624.84 196.85) (xy 702.31 196.85)
-		)
-		(stroke
-			(width 0)
-			(type default)
-		)
-	)
-	(wire
-		(pts
 			(xy 35.56 49.53) (xy 41.91 49.53)
 		)
@@
 	(wire
 		(pts
+			(xy 624.84 196.85) (xy 702.31 196.85)
+		)
+		(stroke
+			(width 0)
+			(type default)
+		)
+	)
+	(wire
+		(pts
 			(xy 650.24 204.47) (xy 702.31 204.47)
 		)
@@
 	(bus
 		(pts
-			(xy 622.3 88.9) (xy 622.3 129.54)
+			(xy 622.3 88.9) (xy 622.3 99.06)
 		)
 		(stroke
@@
 	(wire
 		(pts
+			(xy 676.91 102.87) (xy 702.31 102.87)
+		)
+		(stroke
+			(width 0)
+			(type default)
+		)
+	)
+	(wire
+		(pts
 			(xy 787.4 62.23) (xy 787.4 59.69)
 		)
@@
 	(wire
 		(pts
+			(xy 624.84 153.67) (xy 647.7 153.67)
+		)
+		(stroke
+			(width 0)
+			(type default)
+		)
+	)
+	(wire
+		(pts
 			(xy 346.71 62.23) (xy 346.71 59.69)
 		)
@@
 		)
 	)
+	(bus
+		(pts
+			(xy 622.3 151.13) (xy 622.3 156.21)
+		)
+		(stroke
+			(width 0)
+			(type default)
+		)
+	)
 	(wire
 		(pts
@@
 		)
 	)
+	(wire
+		(pts
+			(xy 624.84 101.6) (xy 676.91 101.6)
+		)
+		(stroke
+			(width 0)
+			(type default)
+		)
+	)
 	(bus
 		(pts
@@
 		)
 	)
+	(label "DDR_DQM0"
+		(at 702.31 153.67 180)
+		(effects
+			(font
+				(size 1.27 1.27)
+			)
+			(justify right bottom)
+		)
+	)
+	(label "DDR_DQS0-"
+		(at 702.31 196.85 180)
+		(effects
+			(font
+				(size 1.27 1.27)
+			)
+			(justify right bottom)
+		)
+	)
 	(label "DDR_BA2"
 		(at 702.31 143.51 180)
@@
 		)
 	)
+	(label "DDR_DQ11"
+		(at 702.31 161.29 180)
+		(effects
+			(font
+				(size 1.27 1.27)
+			)
+			(justify right bottom)
+		)
+	)
 	(label "DDR_DQS0+"
 		(at 702.31 194.31 180)
@@
 		)
 	)
+	(label "DDR_DQ3"
+		(at 702.31 102.87 180)
+		(effects
+			(font
+				(size 1.27 1.27)
+			)
+			(justify right bottom)
+		)
+	)
 	(label "DDR_A14"
 		(at 702.31 125.73 180)
@@
 		)
 	)
-	(label "DDR_DQS1-"
-		(at 702.31 196.85 180)
-		(effects
-			(font
-				(size 1.27 1.27)
-			)
-			(justify right bottom)
-		)
-	)
 	(label "QSPI_DQ2"
 		(at 140.97 97.79 180)
@@
 		(effects
 			(font
-				(size 1.27 1.27)
-			)
-			(justify right bottom)
-		)
-	)
-	(label "DDR_DQ1"
-		(at 702.31 161.29 180)
-		(effects
-			(font

Commit message: 5th time routing is the charm EHH :D
Connections:
- net DDR_A10: no longer U1.AB8 (IO_L22N_T3_34)
- net DDR_A12: no longer U1.Y6 (IO_L18P_T2_34)
- net DDR_CKE: no longer U1.W5 (IO_L15N_T2_DQS_34)
- net DDR_CLK+: now also U1.Y3 (IO_L9P_T1_DQS_34); no longer U1.Y8 (IO_L23P_T3_34)
- net DDR_CLK-: now also U1.AA3 (IO_L9N_T1_DQS_34); no longer U1.Y7 (IO_L23N_T3_34)
- net DDR_DQ2: no longer U1.AA5 (IO_L10P_T1_34)
- net DDR_DQ3: no longer U1.R3 (IO_L3P_T0_DQS_34)
- net DDR_DQ9: no longer U1.V4 (IO_L12P_T1_MRCC_34)
- net DDR_DQS1+: now also U1.Y8 (IO_L23P_T3_34); no longer U1.Y3 (IO_L9P_T1_DQS_34)
- net DDR_DQS1-: now also U1.Y7 (IO_L23N_T3_34); no longer U1.AA3 (IO_L9N_T1_DQS_34)
- net ~{DDR_CAS}: no longer U1.V5 (IO_L16N_T2_34)
- net ~{DDR_RAS}: no longer U1.T4 (IO_L13N_T2_MRCC_34)
- net DDR_A14: no longer names the net of U1.AB1 (IO_L7N_T1_34)
- no-connect marks 12 -> 13
Other:
- note added: "ADDRESS"
- note added: "Data"
- note removed: "Sus A14 >"
