File: PCB/banks.kicad_sch (KiCad schematic)
At the start: 50 parts, among them U1 XC7A50T-FGG484, Y3 100MHz

Commit message: BANNNG
Connections:
- net DDR_DQ10 is gone; now on net DDR_DQS1+: U1.W6 (IO_L15P_T2_DQS_34)
- net DDR_DQ9 is gone; now on net DDR_DQS1-: U1.W5 (IO_L15N_T2_DQS_34)
- net DDR_DQS1+: no longer U1.Y8 (IO_L23P_T3_34)
- net DDR_DQS1-: no longer U1.Y7 (IO_L23N_T3_34)
Changed lines of the file:
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@@
-		)
-	)
-	(label "DDR_DQ9"
-		(at 702.31 166.37 180)
-		(effects
-			(font
-				(size 1.27 1.27)
-			)
-			(justify right bottom)
 		)
 	)
@@
 		)
 	)
+	(label "DDR_DQS1-"
+		(at 702.31 166.37 180)
+		(effects
+			(font
+				(size 1.27 1.27)
+			)
+			(justify right bottom)
+		)
+	)
 	(label "DDR_DQ11"
 		(at 702.31 186.69 180)
@@
 		)
 	)
+	(label "DDR_DQS1+"
+		(at 702.31 163.83 180)
+		(effects
+			(font
+				(size 1.27 1.27)
+			)
+			(justify right bottom)
+		)
+	)
 	(label "DDR_DQS0+"
 		(at 702.31 194.31 180)
@@
 		)
 	)
-	(label "DDR_DQ10"
-		(at 702.31 163.83 180)
-		(effects
-			(font
-				(size 1.27 1.27)
-			)
-			(justify right bottom)
-		)
-	)
 	(label "DDR_A7"
 		(at 702.31 107.95 180)
@@
 		)
 	)
-	(label "DDR_DQS1-"
-		(at 702.31 207.01 180)
-		(effects
-			(font
-				(size 1.27 1.27)
-			)
-			(justify right bottom)
-		)
-	)
 	(label "~{DDR_ODT}"
 		(at 702.31 100.33 180)
@@
 		(effects
 			(font
-				(size 1.27 1.27)
-			)
-			(justify right bottom)
-		)
-	)
-	(label "DDR_DQS1+"
-		(at 702.31 204.47 180)
-		(effects
-			(font

Commit message: KFNESIFHESKJFHSEKJFH UI DID IT
Connections:
- net DDR_DQ8: now also U1.Y7 (IO_L23N_T3_34); no longer U1.Y6 (IO_L18P_T2_34)
- net DDR_DQ9: now reaches U1.AB8 (IO_L22N_T3_34)
- net DDR_DQ10: now reaches U1.Y8 (IO_L23P_T3_34)
Changed lines of the file:
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@@
 	)
 	(no_connect
+		(at 702.31 179.07)
+	)
+	(no_connect
 		(at 261.62 209.55)
 	)
@@
 	)
 	(no_connect
-		(at 702.31 201.93)
-	)
-	(no_connect
 		(at 127 105.41)
 	)
@@
 	)
 	(bus_entry
+		(at 622.3 201.93)
+		(size 2.54 2.54)
+		(stroke
+			(width 0)
+			(type default)
+		)
+	)
+	(bus_entry
+		(at 622.3 204.47)
+		(size 2.54 2.54)
+		(stroke
+			(width 0)
+			(type default)
+		)
+	)
+	(bus_entry
 		(at 622.3 173.99)
 		(size 2.54 2.54)
@@
 	)
 	(bus_entry
-		(at 622.3 176.53)
-		(size 2.54 2.54)
+		(at 142.24 100.33)
+		(size 2.54 -2.54)
 		(stroke
 			(width 0)
@@
 	)
 	(bus_entry
-		(at 142.24 100.33)
-		(size 2.54 -2.54)
+		(at 622.3 199.39)
+		(size 2.54 2.54)
 		(stroke
 			(width 0)
@@
 		)
 	)
+	(bus
+		(pts
+			(xy 622.3 199.39) (xy 622.3 201.93)
+		)
+		(stroke
+			(width 0)
+			(type default)
+		)
+	)
 	(wire
 		(pts
@@
 	(wire
 		(pts
+			(xy 624.84 201.93) (xy 702.31 201.93)
+		)
+		(stroke
+			(width 0)
+			(type default)
+		)
+	)
+	(wire
+		(pts
 			(xy 154.94 149.86) (xy 146.05 149.86)
 		)
@@
 	(bus
 		(pts
-			(xy 622.3 196.85) (xy 622.3 201.93)
+			(xy 622.3 196.85) (xy 622.3 199.39)
 		)
 		(stroke
@@
 	(wire
 		(pts
-			(xy 624.84 204.47) (xy 702.31 204.47)
+			(xy 300.99 49.53) (xy 308.61 49.53)
 		)
 		(stroke
@@
 	(wire
 		(pts
-			(xy 300.99 49.53) (xy 308.61 49.53)
+			(xy 624.84 186.69) (xy 702.31 186.69)
 		)
 		(stroke
@@
 	(wire
 		(pts
-			(xy 624.84 186.69) (xy 702.31 186.69)
+			(xy 300.99 62.23) (xy 300.99 59.69)
 		)
 		(stroke
@@
 		)
 	)
-	(wire
+	(bus
 		(pts
-			(xy 300.99 62.23) (xy 300.99 59.69)
+			(xy 182.88 154.94) (xy 179.07 154.94)
 		)
 		(stroke
@@
 		)
 	)
-	(bus
+	(wire
 		(pts
-			(xy 182.88 154.94) (xy 179.07 154.94)
+			(xy 361.95 49.53) (xy 361.95 52.07)
 		)
 		(stroke
@@
 	(wire
 		(pts
-			(xy 361.95 49.53) (xy 361.95 52.07)
+			(xy 624.84 207.01) (xy 702.31 207.01)
 		)
 		(stroke
@@
 		)
 	)
-	(bus
-		(pts
-			(xy 622.3 173.99) (xy 622.3 176.53)
-		)
-		(stroke
-			(width 0)
-			(type default)
-		)
-	)
 	(wire
 		(pts
@@
 	(wire
 		(pts
-			(xy 624.84 179.07) (xy 702.31 179.07)
-		)
-		(stroke
-			(width 0)
-			(type default)
-		)
-	)
-	(wire
-		(pts
 			(xy 146.05 149.86) (xy 146.05 151.13)
 		)
@@
 	(bus
 		(pts
-			(xy 622.3 176.53) (xy 622.3 179.07)
+			(xy 622.3 173.99) (xy 622.3 179.07)
 		)
 		(stroke
@@
 	(wire
 		(pts
-			(xy 624.84 207.01) (xy 702.31 207.01)
-		)
-		(stroke
-			(width 0)
-			(type default)
-		)
-	)
-	(wire
-		(pts
 			(xy 154.94 158.75) (xy 154.94 163.83)
 		)
@@
 	(wire
 		(pts
+			(xy 624.84 204.47) (xy 702.31 204.47)
+		)
+		(stroke
+			(width 0)
+			(type default)
+		)
+	)
+	(wire
+		(pts
 			(xy 285.75 62.23) (xy 285.75 59.69)
 		)
@@
 		)
 	)
-	(label "DDR_DQ8"
-		(at 702.31 179.07 180)
-		(effects
-			(font
-				(size 1.27 1.27)
-			)
-			(justify right bottom)
-		)
-	)
 	(label "DDR_A11"
 		(at 702.31 115.57 180)
@@
 		)
 	)
+	(label "DDR_DQ8"
+		(at 702.31 207.01 180)
+		(effects
+			(font
+				(size 1.27 1.27)
+			)
+			(justify right bottom)
+		)
+	)
 	(label "DDR_DQ4"
 		(at 702.31 158.75 180)
@@
 		)
 	)
+	(label "DDR_DQ10"
+		(at 702.31 204.47 180)
+		(effects
+			(font
+				(size 1.27 1.27)
+			)
+			(justify right bottom)
+		)
+	)
 	(label "DDR_DQ11"
 		(at 702.31 186.69 180)
@@
 		(effects
 			(font
+				(size 1.27 1.27)
+			)
+			(justify right bottom)
+		)
+	)
+	(label "DDR_DQ9"
+		(at 702.31 201.93 180)
+		(effects
+			(font

Commit message: I'MMMMM crashing out
Connections:
- net DDR_DQS0+: now also U1.W6 (IO_L15P_T2_DQS_34); no longer U1.V9 (IO_L21P_T3_DQS_34)
- net DDR_DQS0-: now also U1.W5 (IO_L15N_T2_DQS_34); no longer U1.V8 (IO_L21N_T3_DQS_34)
- net DDR_DQS1+: now also U1.V9 (IO_L21P_T3_DQS_34); no longer U1.W6 (IO_L15P_T2_DQS_34)
- net DDR_DQS1-: now also U1.V8 (IO_L21N_T3_DQS_34); no longer U1.W5 (IO_L15N_T2_DQS_34)
Changed lines of the file:
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@@
+		)
+	)
+	(label "DDR_DQS1+"
+		(at 702.31 194.31 180)
+		(effects
+			(font
+				(size 1.27 1.27)
+			)
+			(justify right bottom)
 		)
 	)
@@
 		)
 	)
+	(label "DDR_DQS0+"
+		(at 702.31 163.83 180)
+		(effects
+			(font
+				(size 1.27 1.27)
+			)
+			(justify right bottom)
+		)
+	)
 	(label "DDR_DQ8"
 		(at 702.31 207.01 180)
@@
 		)
 	)
-	(label "DDR_DQS1-"
-		(at 702.31 166.37 180)
-		(effects
-			(font
-				(size 1.27 1.27)
-			)
-			(justify right bottom)
-		)
-	)
 	(label "DDR_DQ10"
 		(at 702.31 204.47 180)
@@
 		)
 	)
-	(label "DDR_DQS0-"
-		(at 702.31 196.85 180)
-		(effects
-			(font
-				(size 1.27 1.27)
-			)
-			(justify right bottom)
-		)
-	)
 	(label "DDR_DQ13"
 		(at 702.31 181.61 180)
@@
 		)
 	)
-	(label "DDR_DQS1+"
-		(at 702.31 163.83 180)
-		(effects
-			(font
-				(size 1.27 1.27)
-			)
-			(justify right bottom)
-		)
-	)
-	(label "DDR_DQS0+"
-		(at 702.31 194.31 180)
-		(effects
-			(font
-				(size 1.27 1.27)
-			)
-			(justify right bottom)
-		)
-	)
 	(label "DDR_A4"
 		(at 702.31 97.79 180)
@@
 		)
 	)
+	(label "DDR_DQS0-"
+		(at 702.31 166.37 180)
+		(effects
+			(font
+				(size 1.27 1.27)
+			)
+			(justify right bottom)
+		)
+	)
 	(label "CLK_100MHz"
 		(at 133.35 262.89 180)
@@
 		(effects
 			(font
+				(size 1.27 1.27)
+			)
+			(justify right bottom)
+		)
+	)
+	(label "DDR_DQS1-"
+		(at 702.31 196.85 180)
+		(effects
+			(font

Commit message: GOD TIER DQS pair layer switch to reduce reflections
Connections:
- net DDR_DQ13: now also U1.AB6 (IO_L20N_T3_34); no longer U1.AA6 (IO_L18N_T2_34)
- net DDR_DQ2: now also U1.AA6 (IO_L18N_T2_34); no longer U1.AB6 (IO_L20N_T3_34)
Changed lines of the file:
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@@
-		)
-	)
-	(label "DDR_DQ2"
-		(at 702.31 191.77 180)
-		(effects
-			(font
-				(size 1.27 1.27)
-			)
-			(justify right bottom)
 		)
 	)
@@
 		)
 	)
-	(label "DDR_DQ13"
-		(at 702.31 181.61 180)
-		(effects
-			(font
-				(size 1.27 1.27)
-			)
-			(justify right bottom)
-		)
-	)
 	(label "DDR_A8"
 		(at 702.31 105.41 180)
@@
 		)
 	)
+	(label "DDR_DQ13"
+		(at 702.31 191.77 180)
+		(effects
+			(font
+				(size 1.27 1.27)
+			)
+			(justify right bottom)
+		)
+	)
 	(label "DDR_A9"
 		(at 702.31 125.73 180)
@@
 		(effects
 			(font
+				(size 1.27 1.27)
+			)
+			(justify right bottom)
+		)
+	)
+	(label "DDR_DQ2"
+		(at 702.31 181.61 180)
+		(effects
+			(font

Commit message: I THINK I DID IT
Connections:
- net DDR_DQ0: now also U1.Y6 (IO_L18P_T2_34); no longer U1.W9 (IO_L24P_T3_34)
- net DDR_DQ13: now also U1.AB7 (IO_L20P_T3_34); no longer U1.AB6 (IO_L20N_T3_34)
- net DDR_DQ14: now also U1.AB6 (IO_L20N_T3_34); no longer U1.AA8 (IO_L22P_T3_34)
- net DDR_DQ15: now also U1.AA8 (IO_L22P_T3_34); no longer U1.AB7 (IO_L20P_T3_34)
Changed lines of the file:
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@@
 	)
 	(no_connect
-		(at 702.31 179.07)
-	)
-	(no_connect
 		(at 261.62 209.55)
 	)
@@
 	)
 	(no_connect
+		(at 702.31 209.55)
+	)
+	(no_connect
 		(at 127 113.03)
 	)
@@
 	)
 	(bus_entry
+		(at 622.3 176.53)
+		(size 2.54 2.54)
+		(stroke
+			(width 0)
+			(type default)
+		)
+	)
+	(bus_entry
 		(at 674.37 148.59)
 		(size 2.54 2.54)
@@
 	)
 	(bus_entry
-		(at 622.3 207.01)
-		(size 2.54 2.54)
-		(stroke
-			(width 0)
-			(type default)
-		)
-	)
-	(bus_entry
 		(at 674.37 113.03)
 		(size 2.54 2.54)
@@
 	(bus
 		(pts
+			(xy 622.3 176.53) (xy 622.3 179.07)
+		)
+		(stroke
+			(width 0)
+			(type default)
+		)
+	)
+	(bus
+		(pts
 			(xy 622.3 196.85) (xy 622.3 199.39)
 		)
@@
 		)
 	)
-	(wire
-		(pts
-			(xy 624.84 209.55) (xy 702.31 209.55)
-		)
-		(stroke
-			(width 0)
-			(type default)
-		)
-	)
 	(bus
 		(pts
@@
 	(bus
 		(pts
-			(xy 622.3 173.99) (xy 622.3 179.07)
+			(xy 622.3 173.99) (xy 622.3 176.53)
 		)
 		(stroke
@@
 	(wire
 		(pts
+			(xy 624.84 179.07) (xy 702.31 179.07)
+		)
+		(stroke
+			(width 0)
+			(type default)
+		)
+	)
+	(wire
+		(pts
 			(xy 664.21 119.38) (xy 676.91 119.38)
 		)
@@
 	(bus
 		(pts
-			(xy 622.3 207.01) (xy 622.3 209.55)
+			(xy 622.3 204.47) (xy 622.3 209.55)
 		)
 		(stroke
@@
 		)
 	)
-	(bus
-		(pts
-			(xy 622.3 204.47) (xy 622.3 207.01)
-		)
-		(stroke
-			(width 0)
-			(type default)
-		)
-	)
 	(wire
 		(pts
@@
 		)
 	)
+	(label "DDR_DQ15"
+		(at 702.31 199.39 180)
+		(effects
+			(font
+				(size 1.27 1.27)
+			)
+			(justify right bottom)
+		)
+	)
 	(label "DDR_A11"
 		(at 702.31 115.57 180)
@@
 		)
 	)
-	(label "DDR_DQ15"
-		(at 702.31 189.23 180)
+	(label "DDR_DQ0"
+		(at 702.31 179.07 180)
 		(effects
 			(font
@@
 		)
 	)
-	(label "DDR_DQ14"
-		(at 702.31 199.39 180)
-		(effects
-			(font
-				(size 1.27 1.27)
-			)
-			(justify right bottom)
-		)
-	)
 	(label "DDR_A12"
 		(at 702.31 118.11 180)
@@
 		)
 	)
-	(label "DDR_DQ13"
-		(at 702.31 191.77 180)
-		(effects
-			(font
-				(size 1.27 1.27)
-			)
-			(justify right bottom)
-		)
-	)
 	(label "DDR_A9"
 		(at 702.31 125.73 180)
@@
 		)
 	)
+	(label "DDR_DQ14"
+		(at 702.31 191.77 180)
+		(effects
+			(font
+				(size 1.27 1.27)
+			)
+			(justify right bottom)
+		)
+	)
 	(label "DDR_DQ5"
 		(at 702.31 173.99 180)
@@
 		)
 	)
+	(label "DDR_DQ13"
+		(at 702.31 189.23 180)
+		(effects
+			(font
+				(size 1.27 1.27)
+			)
+			(justify right bottom)
+		)
+	)
 	(label "DDR_A7"
 		(at 702.31 107.95 180)
@@
 		(effects
 			(font
-				(size 1.27 1.27)
-			)
-			(justify right bottom)
-		)
-	)
-	(label "DDR_DQ0"
-		(at 702.31 209.55 180)
-		(effects
-			(font

Commit message: OKAY THIS SHOULD ACTUALLY BE GOOD NOW
Connections:
- net DDR_BA2: now also U1.AB2 (IO_L8N_T1_34); no longer U1.T3 (IO_0_34)
- net DDR_DQ11: now also U1.W9 (IO_L24P_T3_34); no longer U1.W7 (IO_L19N_T3_VREF_34)
- net DDR_DQ14: now also U1.W7 (IO_L19N_T3_VREF_34); no longer U1.AB6 (IO_L20N_T3_34)
- net ~{DDR_RESET}: now also U1.T3 (IO_0_34); no longer U1.AB2 (IO_L8N_T1_34)
Changed lines of the file:
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@@
 	)
 	(no_connect
+		(at 702.31 191.77)
+	)
+	(no_connect
 		(at 702.31 171.45)
 	)
@@
 	)
 	(no_connect
-		(at 702.31 209.55)
-	)
-	(no_connect
 		(at 127 113.03)
 	)
@@
 	)
 	(bus_entry
+		(at 622.3 207.01)
+		(size 2.54 2.54)
+		(stroke
+			(width 0)
+			(type default)
+		)
+	)
+	(bus_entry
 		(at 622.3 156.21)
 		(size 2.54 2.54)
@@
 	)
 	(bus_entry
-		(at 622.3 184.15)
-		(size 2.54 2.54)
-		(stroke
-			(width 0)
-			(type default)
-		)
-	)
-	(bus_entry
 		(at 674.37 115.57)
 		(size 2.54 2.54)
@@
 	)
 	(bus_entry
+		(at 622.3 184.15)
+		(size 2.54 2.54)
+		(stroke
+			(width 0)
+			(type default)
+		)
+	)
+	(bus_entry
 		(at 622.3 153.67)
 		(size 2.54 2.54)
@@
 	)
 	(bus_entry
-		(at 622.3 189.23)
-		(size 2.54 2.54)
-		(stroke
-			(width 0)
-			(type default)
-		)
-	)
-	(bus_entry
 		(at 674.37 113.03)
 		(size 2.54 2.54)
@@
 	(bus
 		(pts
-			(xy 622.3 184.15) (xy 622.3 186.69)
+			(xy 622.3 181.61) (xy 622.3 184.15)
 		)
 		(stroke
@@
 	(wire
 		(pts
-			(xy 624.84 191.77) (xy 702.31 191.77)
-		)
-		(stroke
-			(width 0)
-			(type default)
-		)
-	)
-	(wire
-		(pts
 			(xy 676.91 105.41) (xy 702.31 105.41)
 		)
@@
 		)
 	)
+	(bus
+		(pts
+			(xy 622.3 207.01) (xy 622.3 209.55)
+		)
+		(stroke
+			(width 0)
+			(type default)
+		)
+	)
 	(wire
 		(pts
@@
 		)
 	)
+	(bus
+		(pts
+			(xy 622.3 184.15) (xy 622.3 186.69)
+		)
+		(stroke
+			(width 0)
+			(type default)
+		)
+	)
 	(wire
 		(pts
@@
 	(wire
 		(pts
+			(xy 624.84 209.55) (xy 702.31 209.55)
+		)
+		(stroke
+			(width 0)
+			(type default)
+		)
+	)
+	(wire
+		(pts
 			(xy 354.33 49.53) (xy 361.95 49.53)
 		)
@@
 	(wire
 		(pts
-			(xy 624.84 186.69) (xy 702.31 186.69)
-		)
-		(stroke
-			(width 0)
-			(type default)
-		)
-	)
-	(wire
-		(pts
 			(xy 300.99 62.23) (xy 300.99 59.69)
 		)
@@
 	(wire
 		(pts
-			(xy 111.76 68.58) (xy 109.22 68.58)
+			(xy 624.84 186.69) (xy 702.31 186.69)
 		)
 		(stroke
@@
 	(wire
 		(pts
-			(xy 148.59 49.53) (xy 156.21 49.53)
+			(xy 111.76 68.58) (xy 109.22 68.58)
 		)
 		(stroke
@@
 	(wire
 		(pts
-			(xy 300.99 62.23) (xy 308.61 62.23)
+			(xy 148.59 49.53) (xy 156.21 49.53)
 		)
 		(stroke
@@
 	(wire
 		(pts
-			(xy 712.47 68.58) (xy 712.47 69.85)
+			(xy 300.99 62.23) (xy 308.61 62.23)
 		)
 		(stroke
@@
 	(wire
 		(pts
-			(xy 148.59 62.23) (xy 156.21 62.23)
+			(xy 712.47 68.58) (xy 712.47 69.85)
 		)
 		(stroke
@@
 		)
 	)
-	(bus
+	(wire
 		(pts
-			(xy 622.3 173.99) (xy 622.3 176.53)
+			(xy 148.59 62.23) (xy 156.21 62.23)
 		)
 		(stroke
@@
 	(bus
 		(pts
-			(xy 622.3 181.61) (xy 622.3 184.15)
+			(xy 622.3 173.99) (xy 622.3 176.53)
 		)
 		(stroke
@@
 	(bus
 		(pts
-			(xy 622.3 204.47) (xy 622.3 209.55)
+			(xy 622.3 204.47) (xy 622.3 207.01)
 		)
 		(stroke
@@
 		)
 	)
-	(label "DDR_BA2"
-		(at 702.31 90.17 180)
+	(label "DDR_DQ15"
+		(at 702.31 199.39 180)
 		(effects
 			(font
@@
 		)
 	)
-	(label "DDR_DQ15"
-		(at 702.31 199.39 180)
+	(label "DDR_A11"
+		(at 702.31 115.57 180)
 		(effects
 			(font
@@
 		)
 	)
-	(label "DDR_A11"
-		(at 702.31 115.57 180)
+	(label "DDR_DQ11"
+		(at 702.31 209.55 180)
 		(effects
 			(font
@@
 		)
 	)
-	(label "DDR_DQ11"
-		(at 702.31 186.69 180)
-		(effects
-			(font
-				(size 1.27 1.27)
-			)
-			(justify right bottom)
-		)
-	)
 	(label "DDR_BA1"
 		(at 702.31 151.13 180)
@@
 		)
 	)
-	(label "DDR_DQ14"
-		(at 702.31 191.77 180)
+	(label "DDR_DQ5"
+		(at 702.31 173.99 180)
 		(effects
 			(font
@@
 		)
 	)
-	(label "DDR_DQ5"
-		(at 702.31 173.99 180)
+	(label "DDR_A5"
+		(at 702.31 128.27 180)
 		(effects
 			(font
@@
 		)
 	)
-	(label "DDR_A5"
-		(at 702.31 128.27 180)
+	(label "DDR_DQ13"
+		(at 702.31 189.23 180)
 		(effects
 			(font
@@
 		)
 	)
-	(label "DDR_DQ13"
-		(at 702.31 189.23 180)
+	(label "DDR_BA2"
+		(at 702.31 130.81 180)
 		(effects
 			(font
@@
 		)
 	)
+	(label "~{DDR_RESET}"
+		(at 702.31 90.17 180)
+		(effects
+			(font
+				(size 1.27 1.27)
+			)
+			(justify right bottom)
+		)
+	)
 	(label "~{PCIe_CLKREQ}"
 		(at 175.26 163.83 180)
@@
 		)
 	)
+	(label "DDR_DQ14"
+		(at 702.31 186.69 180)
+		(effects
+			(font
+				(size 1.27 1.27)
+			)
+			(justify right bottom)
+		)
+	)
 	(label "DDR_DQS1-"
 		(at 702.31 196.85 180)
@@
 		(effects
 			(font
-				(size 1.27 1.27)
-			)
-			(justify right bottom)
-		)
-	)
-	(label "~{DDR_RESET}"
-		(at 702.31 130.81 180)
-		(effects
-			(font

Commit message: hopping off for now, I think this will come to me in the morning ;)
Connections:
- net DDR_DQ3: now also U1.T4 (IO_L13N_T2_MRCC_34); no longer U1.R4 (IO_L13P_T2_MRCC_34)
- net DDR_DQM0: now also U1.R4 (IO_L13P_T2_MRCC_34); no longer U1.T4 (IO_L13N_T2_MRCC_34)
Changed lines of the file:
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@@
-		)
-	)
-	(label "DDR_DQ3"
-		(at 702.31 153.67 180)
-		(effects
-			(font
-				(size 1.27 1.27)
-			)
-			(justify right bottom)
 		)
 	)
@@
 		)
 	)
+	(label "DDR_DQ3"
+		(at 702.31 156.21 180)
+		(effects
+			(font
+				(size 1.27 1.27)
+			)
+			(justify right bottom)
+		)
+	)
 	(label "DDR_DQS1+"
 		(at 702.31 194.31 180)
@@
 	(label "DDR_A2"
 		(at 702.31 113.03 180)
-		(effects
-			(font
-				(size 1.27 1.27)
-			)
-			(justify right bottom)
-		)
-	)
-	(label "DDR_DQM0"
-		(at 702.31 156.21 180)
 		(effects
 			(font
@@
 		(effects
 			(font
+				(size 1.27 1.27)
+			)
+			(justify right bottom)
+		)
+	)
+	(label "DDR_DQM0"
+		(at 702.31 153.67 180)
+		(effects
+			(font

Commit message: finished organizing the inner layers JHFESJKFHESJKFHES
Connections:
- net DDR_BA0: now also U1.AB2 (IO_L8N_T1_34); no longer U1.AB5 (IO_L10N_T1_34)
- net DDR_BA2: now also U1.AB5 (IO_L10N_T1_34); no longer U1.AB2 (IO_L8N_T1_34)
Changed lines of the file:
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@@
-		)
-	)
-	(label "DDR_BA0"
-		(at 702.31 140.97 180)
-		(effects
-			(font
-				(size 1.27 1.27)
-			)
-			(justify right bottom)
 		)
 	)
@@
 		)
 	)
+	(label "DDR_BA0"
+		(at 702.31 130.81 180)
+		(effects
+			(font
+				(size 1.27 1.27)
+			)
+			(justify right bottom)
+		)
+	)
 	(label "DDR_A3"
 		(at 702.31 110.49 180)
@@
 		)
 	)
-	(label "DDR_BA2"
-		(at 702.31 130.81 180)
-		(effects
-			(font
-				(size 1.27 1.27)
-			)
-			(justify right bottom)
-		)
-	)
 	(label "DDR_A7"
 		(at 702.31 107.95 180)
@@
 		(effects
 			(font
+				(size 1.27 1.27)
+			)
+			(justify right bottom)
+		)
+	)
+	(label "DDR_BA2"
+		(at 702.31 140.97 180)
+		(effects
+			(font
