File: PCB/_autosave-PCB.kicad_pcb (KiCad board)
At the start: 6 copper layers, 22 x 80 mm, 270 parts, among them J1 Bus_M.2_Edge_M, J2 Conn_ARM_SWD_TagConnect_TC2030, J4 TYPE-C-31-M-12, J7 HDMI_D_1.4, SW1 SW_Push, U1 XC7A50T-FGG484, U10 FT2232HQ, U11 MT41J128M16JT-125:K, U12 PCA9306DC1, U14 UCL0524P, U15 UCL0524P, U16 UCL0524P, U17 TPS62132, U2 MAX20029ATIA/V+, U3 TPD2EUSB30, U4 TPD2EUSB30, U5 TPS2121RUXR, U6 TPD2EUSB30, U7 MT25QL128ABA1EW7-0SIT, U9 M93C56-WMN6TP, Y2 12MHz, Y3 100MHz

Commit message: a bunch of wiring
Routing:
- net /Artix 7 Banks/DDR_DQ3: track 33.5 -> 36.1 mm
- net /Artix 7 Banks/DDR_DQM0: track 27.8 -> 29.6 mm
- net /Artix 7 Banks/DDR_BA1: track 22.0 -> 21.4 mm, vias 2 -> 1
Changed lines of the file:
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@@
+	)
+	(segment
+		(start 152.4086 94.9414)
+		(end 152.523238 94.826762)
+		(width 0.1308)
+		(layer "In2.Cu")
+		(net 348)
 	)
 	(segment
@@
 	(segment
 		(start 148.3586 94.9414)
-		(end 149.5 93.8)
+		(end 152.4086 94.9414)
 		(width 0.1308)
 		(layer "In2.Cu")
@@
 	)
 	(segment
+		(start 149.15 93.1)
+		(end 149.4 93.1)
+		(width 0.1862)
+		(layer "B.Cu")
+		(net 359)
+	)
+	(segment
 		(start 141.15 89.6)
 		(end 143.2628 91.7128)
@@
 	)
 	(segment
+		(start 148.297066 92.147066)
+		(end 148.297066 92.445998)
+		(width 0.1862)
+		(layer "B.Cu")
+		(net 359)
+	)
+	(segment
 		(start 146.663203 92.0059)
 		(end 148.1559 92.0059)
@@
 	)
 	(segment
+		(start 149.4 93.1)
+		(end 149.478652 93.178652)
+		(width 0.1862)
+		(layer "B.Cu")
+		(net 359)
+	)
+	(segment
 		(start 138.9 84.9)
 		(end 141.15 87.15)
@@
 	)
 	(segment
+		(start 148.297066 92.445998)
+		(end 148.951068 93.1)
+		(width 0.1862)
+		(layer "B.Cu")
+		(net 359)
+	)
+	(segment
 		(start 148.1559 92.0059)
 		(end 148.297066 92.147066)
+		(width 0.1862)
+		(layer "B.Cu")
+		(net 359)
+	)
+	(segment
+		(start 148.951068 93.1)
+		(end 149.15 93.1)
 		(width 0.1862)
 		(layer "B.Cu")
@@
 		(net 370)
 	)
-	(segment
-		(start 148.25 92.186827)
-		(end 148.550001 92.486828)
-		(width 0.2)
-		(layer "F.Cu")
-		(net 370)
-	)
-	(segment
-		(start 148.25 92)
-		(end 148.25 92.186827)
-		(width 0.2)
-		(layer "F.Cu")
-		(net 370)
-	)
-	(via
-		(at 148.550001 92.486828)
-		(size 0.45)
-		(drill 0.2)
-		(layers "F.Cu" "B.Cu")
-		(net 370)
-	)
