File: PCB/ddr3.kicad_sch (KiCad schematic)
At the start: 34 parts, among them U11 MT41J128M16JT-125:K

Commit message: even more footprints
Parts:
- C110, C86: footprint (none) -> Capacitor_SMD:C_0402_1005Metric
- C85: footprint (none) -> Capacitor_SMD:C_1206_3216Metric
Changed lines of the file:
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@@
 			)
 		)
-		(property "Footprint" ""
+		(property "Footprint" "Capacitor_SMD:C_0402_1005Metric"
 			(at 176.2252 201.93 0)
 			(effects
@@
 			)
 		)
-		(property "Footprint" ""
+		(property "Footprint" "Capacitor_SMD:C_1206_3216Metric"
 			(at 387.0452 128.27 0)
 			(effects
@@
 			)
 		)
-		(property "Footprint" ""
+		(property "Footprint" "Capacitor_SMD:C_0402_1005Metric"
 			(at 176.2252 191.77 0)
 			(effects

Commit message: fixing a bunch of footprints to standardize
Parts:
- C75: footprint Capacitor_SMD:C_0603_1608Metric -> Capacitor_SMD:C_1206_3216Metric
Changed lines of the file:
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@@
 			)
 		)
-		(property "Footprint" "Capacitor_SMD:C_0603_1608Metric"
+		(property "Footprint" "Capacitor_SMD:C_1206_3216Metric"
 			(at 177.4952 128.27 0)
 			(effects

Commit message: fixing my  VREF decoupling, starting to route it!
Parts:
- removed C110, C86: 10n, Capacitor_SMD:C_0402_1005Metric, symbol Device:C
- added C172: 10n, Capacitor_SMD:C_0402_1005Metric, symbol Device:C
- added C57, C58: 100n, Capacitor_SMD:C_0402_1005Metric, symbol Device:C
- renumbered C58 to C110, C57 to C86
Connections:
- net GND: now also C172.2, C57.2, C58.2
- net at C110.1, C13.1, C86.2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: now also C172.1, C57.1, C58.1
Other:
- note removed: "Decoupling as CLOSE AS POSSIBLE to VREF!"
- moved on the sheet: C110, C86, R17, R18

Commit message: fixing my pads
Parts:
- U11: footprint Package_BGA:Micron_FBGA-96_8x14mm_Layout9x16_P0.8mm -> FPGA:FBGA-96_8x14mm_Layout9x16_P0.8mm
Changed lines of the file:
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@@
 			)
 		)
-		(property "Footprint" "Package_BGA:Micron_FBGA-96_8x14mm_Layout9x16_P0.8mm"
+		(property "Footprint" "FPGA:FBGA-96_8x14mm_Layout9x16_P0.8mm"
 			(at 116.84 213.614 0)
 			(effects
@@
 			)
 		)
-		(property "Footprint" "Package_BGA:Micron_FBGA-96_8x14mm_Layout9x16_P0.8mm"
+		(property "Footprint" "FPGA:FBGA-96_8x14mm_Layout9x16_P0.8mm"
 			(at 283.21 186.944 0)
 			(effects

Commit message: modifying DDR3 CS, routing it too
Parts:
- R42: value 100 -> 1k
Changed lines of the file:
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@@
 			)
 		)
-		(property "Value" "100"
+		(property "Value" "1k"
 			(at 92.71 166.37 90)
 			(effects

Commit message: 5th time routing is the charm EHH :D
Connections:
- net DDR_A14: no longer names the net of U11.T7 (A14)
- no-connect marks 0 -> 1
Changed lines of the file:
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@@
 		(color 0 0 0 0)
 	)
+	(no_connect
+		(at 101.6 152.4)
+	)
 	(bus_entry
 		(at 62.23 198.12)
@@
 	)
 	(bus_entry
-		(at 67.31 152.4)
-		(size -2.54 -2.54)
-		(stroke
-			(width 0)
-			(type default)
-		)
-	)
-	(bus_entry
 		(at 146.05 154.94)
 		(size 2.54 -2.54)
@@
 	(bus
 		(pts
-			(xy 64.77 156.21) (xy 64.77 149.86)
+			(xy 64.77 147.32) (xy 64.77 156.21)
 		)
 		(stroke
@@
 	(wire
 		(pts
-			(xy 67.31 152.4) (xy 101.6 152.4)
-		)
-		(stroke
-			(width 0)
-			(type default)
-		)
-	)
-	(wire
-		(pts
 			(xy 359.41 130.81) (xy 350.52 130.81)
 		)
@@
 		)
 	)
-	(bus
-		(pts
-			(xy 64.77 149.86) (xy 64.77 147.32)
-		)
-		(stroke
-			(width 0)
-			(type default)
-		)
-	)
 	(wire
 		(pts
@@
 		)
 	)
-	(label "DDR_A14"
-		(at 67.31 152.4 0)
-		(effects
-			(font
-				(size 1.27 1.27)
-			)
-			(justify left bottom)
-		)
-	)
