File: PCB/usb-c.kicad_sch (KiCad schematic)
At the start: 14 parts, among them J3 TYPE-C-31-M-12, U17 TPS62132, U3 TPD2EUSB30

Commit message: updated PCB refs
Parts:
- renumbered J3 to J4
Changed lines of the file:
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@@
 		(dnp no)
 		(fields_autoplaced yes)
-		(property "Reference" "J3"
+		(property "Reference" "J4"
 			(at 77.47 67.31 0)
 			(effects
@@
 			(project "PCB"
 				(path "/ed0095eb-57a0-4856-9ac4-7b40bd214a3a/17e1ff09-2cf2-4689-8892-3d8b79d81ef3"
-					(reference "J3")
+					(reference "J4")
 					(unit 1)
 				)

Commit message: working on routing USB and JTAG
Connections:
- net USB_DM renamed USB_D-
- net USB_DP renamed USB_D+
