File: PCB/FPGA-power.kicad_sch (KiCad schematic)
At the start: 33 parts, among them U1 XC7A50T-FGG484

Commit message: cleaning up USB-C, switching some of the decoupling and assigning a bunch of footprints
Parts:
- FB1, FB2: footprint (none) -> Inductor_SMD:L_0805_2012Metric
Changed lines of the file:
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@@
 			)
 		)
-		(property "Footprint" ""
+		(property "Footprint" "Inductor_SMD:L_0805_2012Metric"
 			(at 106.68 239.268 90)
 			(effects
@@
 			)
 		)
-		(property "Footprint" ""
+		(property "Footprint" "Inductor_SMD:L_0805_2012Metric"
 			(at 138.43 41.148 90)
 			(effects

Commit message: even more footprints
Parts:
- C34: footprint (none) -> Capacitor_SMD:C_1206_3216Metric
Changed lines of the file:
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@@
 			)
 		)
-		(property "Footprint" ""
+		(property "Footprint" "Capacitor_SMD:C_1206_3216Metric"
 			(at 88.5952 96.52 0)
 			(effects

Commit message: added the basic form factor
Parts:
- C24: footprint (none) -> Capacitor_Tantalum_SMD:CP_EIA-3528-21_Kemet-B; LCSC (none) -> C542287; MPN (none) -> ETPE330MA9GB
Changed lines of the file:
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@@
 			)
 		)
-		(property "Footprint" ""
+		(property "Footprint" "Capacitor_Tantalum_SMD:CP_EIA-3528-21_Kemet-B"
 			(at 321.0052 66.04 0)
 			(effects
@@
 			(at 320.04 62.23 0)
 			(effects
+				(font
+					(size 1.27 1.27)
+				)
+				(hide yes)
+			)
+		)
+		(property "MPN" "ETPE330MA9GB"
+			(at 320.04 62.23 0)
+			(effects
+				(font
+					(size 1.27 1.27)
+				)
+				(hide yes)
+			)
+		)
+		(property "LCSC" "C542287"
+			(at 320.04 62.23 0)
+			(effects

Commit message: adding the proper 100uF caps
Parts:
- C26: footprint Capacitor_SMD:C_0402_1005Metric -> Capacitor_SMD:C_1206_3216Metric; LCSC (none) -> C15008; MPN (none) -> CL31A107MQHNNNE
Changed lines of the file:
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@@
 			)
 		)
-		(property "Footprint" "Capacitor_SMD:C_0402_1005Metric"
+		(property "Footprint" "Capacitor_SMD:C_1206_3216Metric"
 			(at 141.9352 71.12 0)
 			(effects
@@
 			(at 140.97 67.31 0)
 			(effects
+				(font
+					(size 1.27 1.27)
+				)
+				(hide yes)
+			)
+		)
+		(property "MPN" "CL31A107MQHNNNE"
+			(at 140.97 67.31 0)
+			(effects
+				(font
+					(size 1.27 1.27)
+				)
+				(hide yes)
+			)
+		)
+		(property "LCSC" "C15008"
+			(at 140.97 67.31 0)
+			(effects

Commit message: VCCINT decoupling fanout
Parts:
- added C148: 470n, Capacitor_SMD:C_0201_0603Metric, symbol Device:C
Connections:
- net +1V0: now also C148.1
- net GND: now also C148.2
Other:
- moved on the sheet: C21, C22, C23, C24

Commit message: adding return via's and cleaning up the schematic a bit!
Other:
- note added: "Remember to model pi filter!"
- note removed: "Decoupling before and after bead for high current rail!"
Changed lines of the file:
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@@
 		)
 	)
-	(text "Decoupling before and after bead for high current rail!"
+	(text "Remember to model pi filter!"
 		(exclude_from_sim no)
-		(at 107.95 224.79 0)
+		(at 106.934 222.504 0)
 		(effects
 			(font
