File: PCB/power.kicad_sch (KiCad schematic)
At the start: 40 parts, among them U2 MAX20029ATIA/V+, U5 TPS2121RUXR

Commit message: even more footprints
Parts:
- C45, C49, C51, C53: footprint (none) -> Capacitor_SMD:C_1206_3216Metric
- C46, C48, C50, C52: footprint (none) -> Capacitor_SMD:C_0402_1005Metric
Changed lines of the file:
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@@
 			)
 		)
-		(property "Footprint" ""
+		(property "Footprint" "Capacitor_SMD:C_0402_1005Metric"
 			(at 323.5452 148.59 0)
 			(effects
@@
 			)
 		)
-		(property "Footprint" ""
+		(property "Footprint" "Capacitor_SMD:C_1206_3216Metric"
 			(at 343.8652 148.59 0)
 			(effects
@@
 			)
 		)
-		(property "Footprint" ""
+		(property "Footprint" "Capacitor_SMD:C_1206_3216Metric"
 			(at 343.8652 207.01 0)
 			(effects
@@
 			)
 		)
-		(property "Footprint" ""
+		(property "Footprint" "Capacitor_SMD:C_0402_1005Metric"
 			(at 323.5452 177.8 0)
 			(effects
@@
 			)
 		)
-		(property "Footprint" ""
+		(property "Footprint" "Capacitor_SMD:C_0402_1005Metric"
 			(at 323.5452 207.01 0)
 			(effects
@@
 			)
 		)
-		(property "Footprint" ""
+		(property "Footprint" "Capacitor_SMD:C_1206_3216Metric"
 			(at 343.8652 177.8 0)
 			(effects
@@
 			)
 		)
-		(property "Footprint" ""
+		(property "Footprint" "Capacitor_SMD:C_0402_1005Metric"
 			(at 308.3052 86.36 0)
 			(effects
@@
 			)
 		)
-		(property "Footprint" ""
+		(property "Footprint" "Capacitor_SMD:C_1206_3216Metric"
 			(at 313.3852 119.38 0)
 			(effects

Commit message: completely organized the MAX20029 buck and cleaned up some silkscreen
Connections:
- net +1V2: no longer C48.2, R4.2, R5.1, U2.8 (OUTS2)
- net +1V5: no longer C50.2, R6.2, R7.1, U2.14 (OUTS3)
- net +1V8: no longer C52.2, R8.2, R9.1, U2.22 (OUTS4)
- new net: C48.2, R4.2, R5.1, U2.8 (OUTS2)
- new net: C50.2, R6.2, R7.1, U2.14 (OUTS3)
- new net: C52.2, R8.2, R9.1, U2.22 (OUTS4)
Changed lines of the file:
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@@
-	)
-	(junction
-		(at 304.8 198.12)
-		(diameter 0)
-		(color 0 0 0 0)
 	)
 	(junction
@@
 	)
 	(junction
-		(at 304.8 208.28)
-		(diameter 0)
-		(color 0 0 0 0)
-	)
-	(junction
 		(at 289.56 88.9)
 		(diameter 0)
@@
 	)
 	(junction
-		(at 304.8 168.91)
-		(diameter 0)
-		(color 0 0 0 0)
-	)
-	(junction
 		(at 93.98 132.08)
 		(diameter 0)
@@
 	)
 	(junction
-		(at 304.8 149.86)
-		(diameter 0)
-		(color 0 0 0 0)
-	)
-	(junction
 		(at 280.67 76.2)
 		(diameter 0)
@@
 	)
 	(junction
-		(at 304.8 179.07)
-		(diameter 0)
-		(color 0 0 0 0)
-	)
-	(junction
 		(at 312.42 179.07)
 		(diameter 0)
@@
 	)
 	(junction
-		(at 304.8 139.7)
-		(diameter 0)
-		(color 0 0 0 0)
-	)
-	(junction
 		(at 312.42 149.86)
 		(diameter 0)
@@
 	(wire
 		(pts
-			(xy 304.8 149.86) (xy 304.8 139.7)
-		)
-		(stroke
-			(width 0)
-			(type default)
-		)
-	)
-	(wire
-		(pts
 			(xy 298.45 76.2) (xy 307.34 76.2)
 		)
@@
 	(wire
 		(pts
-			(xy 298.45 168.91) (xy 304.8 168.91)
+			(xy 298.45 168.91) (xy 312.42 168.91)
 		)
 		(stroke
@@
 	(wire
 		(pts
-			(xy 304.8 208.28) (xy 304.8 198.12)
-		)
-		(stroke
-			(width 0)
-			(type default)
-		)
-	)
-	(wire
-		(pts
 			(xy 285.75 120.65) (xy 304.8 120.65)
 		)
@@
 	(wire
 		(pts
-			(xy 304.8 198.12) (xy 312.42 198.12)
-		)
-		(stroke
-			(width 0)
-			(type default)
-		)
-	)
-	(wire
-		(pts
 			(xy 322.58 149.86) (xy 312.42 149.86)
 		)
@@
 	(wire
 		(pts
-			(xy 304.8 179.07) (xy 304.8 168.91)
-		)
-		(stroke
-			(width 0)
-			(type default)
-		)
-	)
-	(wire
-		(pts
 			(xy 312.42 149.86) (xy 312.42 148.59)
 		)
@@
 	(wire
 		(pts
-			(xy 285.75 179.07) (xy 304.8 179.07)
+			(xy 285.75 179.07) (xy 312.42 179.07)
 		)
 		(stroke
@@
 	(wire
 		(pts
-			(xy 298.45 139.7) (xy 304.8 139.7)
-		)
-		(stroke
-			(width 0)
-			(type default)
-		)
-	)
-	(wire
-		(pts
 			(xy 251.46 102.87) (xy 251.46 110.49)
 		)
@@
 	(wire
 		(pts
-			(xy 304.8 168.91) (xy 312.42 168.91)
-		)
-		(stroke
-			(width 0)
-			(type default)
-		)
-	)
-	(wire
-		(pts
 			(xy 71.12 165.1) (xy 71.12 167.64)
 		)
@@
 	(wire
 		(pts
-			(xy 312.42 179.07) (xy 304.8 179.07)
-		)
-		(stroke
-			(width 0)
-			(type default)
-		)
-	)
-	(wire
-		(pts
-			(xy 298.45 198.12) (xy 304.8 198.12)
+			(xy 298.45 198.12) (xy 312.42 198.12)
 		)
 		(stroke
@@
 	(wire
 		(pts
-			(xy 285.75 149.86) (xy 304.8 149.86)
-		)
-		(stroke
-			(width 0)
-			(type default)
-		)
-	)
-	(wire
-		(pts
 			(xy 322.58 168.91) (xy 322.58 170.18)
 		)
@@
 	(wire
 		(pts
-			(xy 312.42 208.28) (xy 304.8 208.28)
+			(xy 285.75 208.28) (xy 312.42 208.28)
 		)
 		(stroke
@@
 	(wire
 		(pts
-			(xy 304.8 139.7) (xy 312.42 139.7)
+			(xy 298.45 139.7) (xy 312.42 139.7)
 		)
 		(stroke
@@
 	(wire
 		(pts
-			(xy 312.42 149.86) (xy 304.8 149.86)
+			(xy 285.75 149.86) (xy 312.42 149.86)
 		)
 		(stroke
@@
 		)
 		(stroke
-			(width 0)
-			(type default)
-		)
-	)
-	(wire
-		(pts
-			(xy 285.75 208.28) (xy 304.8 208.28)
-		)
-		(stroke

Commit message: adding return via's and cleaning up the schematic a bit!
Other:
- note added: "Divider: R1 = R2[( VOUT / 1 ) − 1] Frequency compensation: C1 = 15e-12(R2 / R1)"
- note removed: "+VM2_3V3 is the M.2 3.3V power source +VBUS_3V3 is the USB power source, bucked down This circuit ensures that USB doesn't backfeed into the M.2 connector, frying the motherboard, and also prioritizes reliable M.2 connector power if both are plugged in! Switchover is at 3.18V using PR1 voltage divider which is really optimal with 1% resistors because m.2 connector minimum voltage is 3.135V"
- note removed: "Divider: R1 = R2[( VOUT / 1 ) − 1]"
- note removed: "Frequency compensation: C1 = 15e-12(R2 / R1)"
- moved on the sheet: C41, C42, C43, C44, C45, C46, C48, C49, C50, C51, C52, C53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
