File: PCB/PCB.kicad_sch (KiCad schematic)
At the start: 0 parts

Commit message: removing ethernet, out of scope ;)
Other:
- sheet Artix 7 Banks ports: added none; removed {EPHY}
- sheet Ethernet ports: added none; removed {EPHY}
Changed lines of the file:
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@@
-	(bus
-		(pts
-			(xy 228.6 182.88) (xy 228.6 175.26)
-		)
-		(stroke
-			(width 0)
-			(type default)
-		)
-	)
 	(bus
 		(pts
@@
 	(bus
 		(pts
-			(xy 172.72 189.23) (xy 172.72 182.88)
-		)
-		(stroke
-			(width 0)
-			(type default)
-		)
-	)
-	(bus
-		(pts
 			(xy 129.54 147.32) (xy 140.97 147.32)
 		)
@@
 		(pts
 			(xy 134.62 128.27) (xy 201.93 128.27)
-		)
-		(stroke
-			(width 0)
-			(type default)
-		)
-	)
-	(bus
-		(pts
-			(xy 172.72 182.88) (xy 228.6 182.88)
 		)
 		(stroke
@@
 				)
 				(justify left top)
-			)
-		)
-		(pin "{EPHY}" bidirectional
-			(at 172.72 189.23 90)
-			(effects
-				(font
-					(size 1.27 1.27)
-				)
-				(justify right)
 			)
 		)
@@
 			)
 		)
-		(pin "{EPHY}" bidirectional
-			(at 228.6 175.26 270)
-			(effects
-				(font
-					(size 1.27 1.27)
-				)
-				(justify left)
-			)
-		)

Commit message: workingng on organizing the board
Other:
- sheet Ethernet renamed USB to UART
- sheet USB-C and JTAG renamed USB to JTAG
- sheet USB to UART: file ethernet.kicad_sch -> usb-c.kicad_sch
Changed lines of the file:
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@@
 			(color 0 0 0 0.0000)
 		)
-		(property "Sheetname" "Ethernet"
+		(property "Sheetname" "USB to UART"
 			(at 140.97 188.5184 0)
 			(effects
@@
 			)
 		)
-		(property "Sheetfile" "ethernet.kicad_sch"
+		(property "Sheetfile" "usb-c.kicad_sch"
 			(at 140.97 248.2346 0)
 			(effects
@@
 			(color 0 0 0 0.0000)
 		)
-		(property "Sheetname" "USB-C and JTAG"
+		(property "Sheetname" "USB to JTAG"
 			(at 274.32 51.3584 0)
 			(effects

Commit message: cleaning up the schematic
Other:
- removed sheet USB to UART
Changed lines of the file:
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@@
-	)
-	(sheet
-		(at 140.97 189.23)
-		(size 59.69 58.42)
-		(exclude_from_sim no)
-		(in_bom yes)
-		(on_board yes)
-		(dnp no)
-		(fields_autoplaced yes)
-		(stroke
-			(width 0.1524)
-			(type solid)
-		)
-		(fill
-			(color 0 0 0 0.0000)
-		)
-		(property "Sheetname" "USB to UART"
-			(at 140.97 188.5184 0)
-			(effects
-				(font
-					(size 1.27 1.27)
-				)
-				(justify left bottom)
-			)
-		)
-		(property "Sheetfile" "usb-c.kicad_sch"
-			(at 140.97 248.2346 0)
-			(effects
-				(font
-					(size 1.27 1.27)
-				)
-				(justify left top)
-			)
-		)
-		(instances
-			(project "PCB"
-				(path "/ed0095eb-57a0-4856-9ac4-7b40bd214a3a"
-					(page "11")
-				)
-			)
-		)
 	)
 	(sheet

Commit message: cleaned up the schematic to look cooler
Other:
- added sheet USB-C (usb-c.kicad_sch)
- sheet USB to JTAG ports: added {USB}; removed none
Changed lines of the file:
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@@
 	(bus
 		(pts
-			(xy 261.62 139.7) (xy 274.32 139.7)
+			(xy 233.68 175.26) (xy 233.68 189.23)
 		)
 		(stroke
@@
 	(bus
 		(pts
-			(xy 233.68 175.26) (xy 233.68 189.23)
+			(xy 172.72 189.23) (xy 172.72 182.88)
 		)
 		(stroke
@@
 	(bus
 		(pts
+			(xy 237.49 175.26) (xy 237.49 189.23)
+		)
+		(stroke
+			(width 0)
+			(type default)
+		)
+	)
+	(bus
+		(pts
 			(xy 228.6 110.49) (xy 228.6 116.84)
 		)
@@
 	(bus
 		(pts
+			(xy 229.87 175.26) (xy 229.87 189.23)
+		)
+		(stroke
+			(width 0)
+			(type default)
+		)
+	)
+	(bus
+		(pts
 			(xy 129.54 151.13) (xy 201.93 151.13)
 		)
@@
 	(bus
 		(pts
+			(xy 304.8 110.49) (xy 304.8 116.84)
+		)
+		(stroke
+			(width 0)
+			(type default)
+		)
+	)
+	(bus
+		(pts
+			(xy 222.25 182.88) (xy 222.25 175.26)
+		)
+		(stroke
+			(width 0)
+			(type default)
+		)
+	)
+	(bus
+		(pts
 			(xy 233.68 116.84) (xy 233.68 83.82)
 		)
@@
 	(bus
 		(pts
-			(xy 261.62 151.13) (xy 274.32 151.13)
+			(xy 241.3 175.26) (xy 241.3 189.23)
 		)
 		(stroke
@@
 	(bus
 		(pts
-			(xy 261.62 147.32) (xy 274.32 147.32)
+			(xy 172.72 182.88) (xy 222.25 182.88)
 		)
 		(stroke
@@
 		)
 	)
-	(bus
-		(pts
-			(xy 261.62 143.51) (xy 274.32 143.51)
-		)
-		(stroke
-			(width 0)
-			(type default)
+	(sheet
+		(at 274.32 116.84)
+		(size 59.69 58.42)
+		(exclude_from_sim no)
+		(in_bom yes)
+		(on_board yes)
+		(dnp no)
+		(fields_autoplaced yes)
+		(stroke
+			(width 0.1524)
+			(type solid)
+		)
+		(fill
+			(color 0 0 0 0.0000)
+		)
+		(property "Sheetname" "USB-C"
+			(at 274.32 116.1284 0)
+			(effects
+				(font
+					(size 1.27 1.27)
+				)
+				(justify left bottom)
+			)
+		)
+		(property "Sheetfile" "usb-c.kicad_sch"
+			(at 274.32 175.8446 0)
+			(effects
+				(font
+					(size 1.27 1.27)
+				)
+				(justify left top)
+			)
+		)
+		(pin "{USB}" bidirectional
+			(at 304.8 116.84 90)
+			(effects
+				(font
+					(size 1.27 1.27)
+				)
+				(justify right)
+			)
+		)
+		(instances
+			(project "PCB"
+				(path "/ed0095eb-57a0-4856-9ac4-7b40bd214a3a"
+					(page "11")
+				)
+			)
 		)
 	)
@@
 	)
 	(sheet
-		(at 274.32 116.84)
+		(at 201.93 189.23)
 		(size 59.69 58.42)
 		(exclude_from_sim no)
@@
 		)
 		(property "Sheetname" "DDR3"
-			(at 274.32 116.1284 0)
+			(at 201.93 188.5184 0)
 			(effects
 				(font
@@
 		)
 		(property "Sheetfile" "ddr3.kicad_sch"
-			(at 274.32 175.8446 0)
+			(at 201.93 248.2346 0)
 			(effects
 				(font
@@
 		)
 		(pin "{DDR_ADDRESS}" bidirectional
-			(at 274.32 143.51 180)
-			(effects
-				(font
-					(size 1.27 1.27)
-				)
-				(justify left)
+			(at 237.49 189.23 90)
+			(effects
+				(font
+					(size 1.27 1.27)
+				)
+				(justify right)
+			)
+		)
+		(pin "{DDR_CLK}" input
+			(at 233.68 189.23 90)
+			(effects
+				(font
+					(size 1.27 1.27)
+				)
+				(justify right)
 			)
 		)
 		(pin "{DDR_COMMAND}" input
-			(at 274.32 151.13 180)
-			(effects
-				(font
-					(size 1.27 1.27)
-				)
-				(justify left)
+			(at 229.87 189.23 90)
+			(effects
+				(font
+					(size 1.27 1.27)
+				)
+				(justify right)
 			)
 		)
 		(pin "{DDR_DATA}" bidirectional
-			(at 274.32 139.7 180)
-			(effects
-				(font
-					(size 1.27 1.27)
-				)
-				(justify left)
-			)
-		)
-		(pin "{DDR_CLK}" input
-			(at 274.32 147.32 180)
-			(effects
-				(font
-					(size 1.27 1.27)
-				)
-				(justify left)
+			(at 241.3 189.23 90)
+			(effects
+				(font
+					(size 1.27 1.27)
+				)
+				(justify right)
 			)
 		)
@@
 			)
 		)
-		(pin "{DDR_ADDRESS}" bidirectional
-			(at 261.62 143.51 0)
-			(effects
-				(font
-					(size 1.27 1.27)
-				)
-				(justify right)
-			)
-		)
-		(pin "{DDR_CLK}" output
-			(at 261.62 147.32 0)
-			(effects
-				(font
-					(size 1.27 1.27)
-				)
-				(justify right)
-			)
-		)
-		(pin "{DDR_COMMAND}" output
-			(at 261.62 151.13 0)
-			(effects
-				(font
-					(size 1.27 1.27)
-				)
-				(justify right)
-			)
-		)
-		(pin "{DDR_DATA}" bidirectional
-			(at 261.62 139.7 0)
-			(effects
-				(font
-					(size 1.27 1.27)
-				)
-				(justify right)
-			)
-		)
-		(pin "{HDMI}" bidirectional
-			(at 233.68 175.26 270)
-			(effects
-				(font
-					(size 1.27 1.27)
-				)
-				(justify left)
-			)
-		)
 		(pin "BUCK_PG4" input
 			(at 201.93 128.27 180)
@@
 				)
 				(justify right)
+			)
+		)
+		(pin "{DDR_ADDRESS}" bidirectional
+			(at 237.49 175.26 270)
+			(effects
+				(font
+					(size 1.27 1.27)
+				)
+				(justify left)
+			)
+		)
+		(pin "{DDR_CLK}" output
+			(at 233.68 175.26 270)
+			(effects
+				(font
+					(size 1.27 1.27)
+				)
+				(justify left)
+			)
+		)
+		(pin "{DDR_COMMAND}" output
+			(at 229.87 175.26 270)
+			(effects
+				(font
+					(size 1.27 1.27)
+				)
+				(justify left)
+			)
+		)
+		(pin "{DDR_DATA}" bidirectional
+			(at 241.3 175.26 270)
+			(effects
+				(font
+					(size 1.27 1.27)
+				)
+				(justify left)
+			)
+		)
+		(pin "{HDMI}" bidirectional
+			(at 222.25 175.26 270)
+			(effects
+				(font
+					(size 1.27 1.27)
+				)
+				(justify left)
 			)
 		)
@@
 			)
 		)
+		(pin "{USB}" bidirectional
+			(at 304.8 110.49 270)
+			(effects
+				(font
+					(size 1.27 1.27)
+				)
+				(justify left)
+			)
+		)
 		(instances
 			(project "PCB"
@@
 	)
 	(sheet
-		(at 201.93 189.23)
+		(at 140.97 189.23)
 		(size 59.69 58.42)
 		(exclude_from_sim no)
@@
 		)
 		(property "Sheetname" "HDMI"
-			(at 201.93 188.5184 0)
+			(at 140.97 188.5184 0)
 			(effects
 				(font
@@
 		)
 		(property "Sheetfile" "hdmi.kicad_sch"
-			(at 201.93 248.2346 0)
+			(at 140.97 248.2346 0)
 			(effects
 				(font
@@
 		)
 		(pin "{HDMI}" bidirectional
-			(at 233.68 189.23 90)
-			(effects
-				(font
+			(at 172.72 189.23 90)
+			(effects
+				(font

Commit message: heading to the next class, some minor changes
Other:
- note added: "Reviews on: - Reddit - EEBlog - KiCad Discord - Slack"
Changed lines of the file:
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@@
+		)
+	)
+	(text "Reviews on:\n- Reddit\n- EEBlog\n- KiCad Discord\n- Slack"
+		(exclude_from_sim no)
+		(at 16.256 30.734 0)
+		(effects
+			(font
+				(size 1.27 1.27)
+			)
+			(justify left)
 		)
 	)

Commit message: proper DDR3 decoupling!
Other:
- note removed: "For a production board: - make R8, R6, R35 and R33, 0402 and exact! - make 47nF caps 0402"
- note removed: "Reviews on: - Reddit - EEBlog - KiCad Discord - Slack"
Changed lines of the file:
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@@
 		(comment 1 "https://github.com/KaiPereira/M.2-FPGA-Accelerator")
 	)
-	(text "For a production board: \n- make R8, R6, R35 and R33, 0402 and exact!\n- make 47nF caps 0402"
+	(text_box "For a production board: \n- make R8, R6, R35 and R33, 0402 and exact!\n- make 47nF caps 0402"
 		(exclude_from_sim no)
-		(at 16.256 18.542 0)
+		(at 25.4 27.94 0)
+		(size 49.53 10.16)
+		(margins 0.9525 0.9525 0.9525 0.9525)
+		(stroke
+			(width 0)
+			(type solid)
+		)
+		(fill
+			(type none)
+		)
 		(effects
 			(font
@@
 		)
 	)
-	(text "Reviews on:\n- Reddit\n- EEBlog\n- KiCad Discord\n- Slack"
+	(text_box "Reviews on:\n- Reddit\n- EEBlog\n- KiCad Discord\n- Slack"
 		(exclude_from_sim no)
-		(at 16.256 30.734 0)
+		(at 25.4 39.37 0)
+		(size 20.32 13.97)
+		(margins 0.9525 0.9525 0.9525 0.9525)
+		(stroke
+			(width 0)
+			(type solid)
+		)
+		(fill
+			(type none)
+		)
 		(effects
 			(font
